Commit message: Update xacro for real robot

File: rb_theron_description/robots/default.urdf.xacro (robot description, xacro)
@@ -1 +1 @@
-basic.urdf.xacro
+rb_theron.urdf.xacro

File: rb_theron_description/urdf/bases/theron_base.urdf.xacro (robot description, xacro)
@@ -1,5 +1,6 @@
 <?xml version="1.0"?>
 <robot name="theron_base" xmlns:xacro="http://www.ros.org/wiki/xacro">
-  <xacro:macro name="theron_base" params="publish_bf hq">
+  <xacro:macro name="theron_base" params="prefix publish_bf hq">
+    <xacro:include filename="$(find rb_theron_description)/urdf/utils/inertial.urdf.xacro" />
     <xacro:property name="PI" value="3.1415926535897931"/>
     <!-- xacro:property name="wheel_width" value="0.150" / -->
@@ -18,5 +19,5 @@
         <mass value="45" />
         <origin xyz="0.0 0.0 0.0" />
-        <xacro:solid_cuboid_inertia m="45" w="0.3275" h="0.2775" d="0.1525" />
+        <xacro:solid_cuboid_inertia mass="45" width="0.3275" height="0.2775" depth="0.1525" />
       </inertial>
       <visual>

File: rb_theron_description/urdf/ros2_control.urdf.xacro (robot description, xacro)
@@ -1,9 +1,9 @@
 <?xml version="1.0"?>
 <robot xmlns:xacro="http://wiki.ros.org/xacro">
-  <xacro:macro name="ros2_control">
+  <xacro:macro name="ros2_control" params="namespace:=robot config_controllers:=''">
       <gazebo>
         <plugin name="ros_control" filename="libgazebo_ros2_control.so">
-          <namespace>$(arg robot_id)</namespace>
-          <parameters>$(arg config_controllers)</parameters>
+          <namespace>${namespace}</namespace>
+          <parameters>${config_controllers}</parameters>
         </plugin>
       </gazebo>
