Commit message: Optimize simulation for omnitheron

File: rb_theron_description/robots/rb_theron_omni.urdf.xacro (robot description, xacro)
@@ -1,54 +1,91 @@
 <?xml version="1.0"?>
-<robot name="rb_theron"
-	xmlns:xacro="http://www.ros.org/wiki/xacro">
-	<!-- ***************** -->
-	<!-- Imported elements -->
-	<!-- ***************** -->
-	<!-- First we import all posible elements defined in the urdf.xacro files. All these elements are defined as macro:xacros -->
-	<!-- Import differential base elements -->
-	<xacro:include filename="$(find rb_theron_description)/robots/rb_theron_base_omni.urdf.xacro" />
-	<!-- Import wheels -->
-	<xacro:include filename="$(find rb_theron_description)/urdf/wheels/omni_wheel.urdf.xacro" />
-	<!-- Import all available sensors -->
-	<xacro:include filename="$(find robotnik_sensors)/urdf/all_sensors.urdf.xacro" />
-	<!-- Import Gazebo Stuff -->
-	<xacro:include filename="$(find rb_theron_description)/urdf/common.gazebo.xacro" />
-	<!-- ***************** -->
-	<!-- Global parameters -->
-	<!-- ***************** -->
-	<xacro:property name="PI" value="3.1415926535897931"/>
-	<!-- Wheel parameters -->
-	<!--xacro:property name="wheel_offset_x" value="0" />
-	<xacro:property name="wheel_offset_y" value="0.2516" />
-	<xacro:property name="wheel_offset_z" value="0.0" /-->
-	<!-- Flag to select the high or low quality model -->
-	<xacro:property name="hq" value="true" />
-	<!-- *************** -->
-	<!-- Robots Elements -->
-	<!-- *************** -->
-	<xacro:arg name="prefix" default="robot_"/>
-	<xacro:arg name="gpu" default="true"/>
-	<!-- Here we create the robot elements using the xacro:macros imported at the beggining of this file -->
-	<!-- base with wheels -->
-	<xacro:rb_theron_base prefix="$(arg prefix)" hq="${hq}" />
-	<!-- Gazebo ros control pluggins -->
-	<xacro:ros_control/>
-	<xacro:gazebo_colors prefix="$(arg prefix)"/>
-  <!-- SENSORS -->
-  <!-- TODO: Moved 0.01 in x, otherwise the camera is still inside the robot -->
-	<xacro:sensor_orbbec_astra prefix="$(arg prefix)front_rgbd_camera" parent="$(arg prefix)base_link" prefix_topic="front_rgbd_camera">
-		<origin xyz="0.3305 0.0 0.1748" rpy="0 0 0"/>
-	</xacro:sensor_orbbec_astra>
-	<xacro:sensor_imu_hector prefix="$(arg prefix)imu" parent="$(arg prefix)base_link">
-		<origin xyz="-0.1975 0.0 0.1598" rpy="0 0 0"/>
-	</xacro:sensor_imu_hector>
-	<!--xacro:sensor_sick_nanoscan3 prefix="$(arg prefix)front_laser" parent="$(arg prefix)base_link" prefix_topic="front_laser" min_angle="-2.0507619" max_angle="2.0507619">
-		<origin xyz="0.250 0.0 0.1643" rpy="0 3.1416 3.1416"/>
-	</xacro:sensor_sick_nanoscan3-->
-	<xacro:sensor_sick_tim571 prefix="$(arg prefix)front_laser" parent="$(arg prefix)base_link" prefix_topic="front_laser" min_angle="-2.0507619" max_angle="2.0507619" gpu="$(arg gpu)">
-		<origin xyz="0.2675 -0.215 0.1613" rpy="0 -3.1416 2.3562"/>
-	</xacro:sensor_sick_tim571>
-	<xacro:sensor_sick_tim571 prefix="$(arg prefix)rear_laser" parent="$(arg prefix)base_link" prefix_topic="rear_laser" min_angle="-2.0507619" max_angle="2.0507619" gpu="$(arg gpu)">
-		<origin xyz="-0.2675 0.215 0.1613" rpy="0 -3.1416 -0.7854"/>
-	</xacro:sensor_sick_tim571>
+<robot name="rbkairos" xmlns:xacro="http://wiki.ros.org/xacro">
+  <!-- ***************** -->
+  <!-- Imported elements -->
+  <!-- ***************** -->
+  <!-- First we import all posible elements defined in the urdf.xacro files. All these elements are defined as macro:xacros -->
+  <!-- Import rb_theron_omni base elements -->
+  <xacro:include filename="$(find rb_theron_description)/urdf/bases/rb_theron_omni_base.urdf.xacro" />
+  <!-- Import rb_theron_omni wheels -->
+  <xacro:include filename="$(find rb_theron_description)/urdf/wheels/omni_wheel.urdf.xacro" />
+  <!-- Import all available sensors -->
+  <xacro:include filename="$(find robotnik_sensors)/urdf/all_sensors.urdf.xacro" />
+  <!-- Flag to select the high or low quality model -->
+  <xacro:property name="hq" value="true" />
+  <xacro:arg name="prefix" default="robot_"/>
+  <xacro:arg name="ros_planar_move_plugin" default="false"/>
+  <xacro:arg name="load_kinematics_file" default="false"/> <!-- Necesarry for ur_description compatible with official ur drivers-->
+  <xacro:arg name="use_gpu_for_simulation" default="false"/>
+   <xacro:property name="PI" value="3.1415926535897931"/>
+   <!-- Wheel parameters -->
+   <xacro:property name="wheel_offset_x" value="0.2175" />    <!-- x,y,z in translation from base_link to the center of the wheel -->
+   <xacro:property name="wheel_offset_y" value="0.204" />
+   <xacro:property name="wheel_offset_z" value="0.0" />
+   <xacro:property name="front_laser_offset_x" value="0.25109"/>
+   <xacro:property name="front_laser_offset_y" value="-0.19859"/>
+   <xacro:property name="front_laser_offset_z" value="0.1847"/>
+   <xacro:property name="rear_laser_offset_x" value="-0.25109"/>
+   <xacro:property name="rear_laser_offset_y" value="0.19859"/>
+   <xacro:property name="rear_laser_offset_z" value="0.1847"/>
+   <xacro:property name="front_ptz_camera_offset_x" value="0.308"/>
+   <xacro:property name="front_ptz_camera_offset_y" value="0.141"/>
+   <xacro:property name="front_ptz_camera_offset_z" value="0.195"/>
+   <xacro:property name="rear_ptz_camera_offset_x" value="-0.308"/>
+   <xacro:property name="rear_ptz_camera_offset_y" value="-0.141"/>
+   <xacro:property name="rear_ptz_camera_offset_z" value="0.195"/>
+   <xacro:property name="imu_offset_x" value="0.2201"/>
+   <xacro:property name="imu_offset_y" value="0.0855"/>
+   <xacro:property name="imu_offset_z" value="0.0917"/>
+   <xacro:property name="front_rgbd_camera_offset_x" value="0.29545"/>
+   <xacro:property name="front_rgbd_camera_offset_y" value="0.0"/>
+   <xacro:property name="front_rgbd_camera_offset_z" value="0.1662"/>
+ <xacro:property name="rear_rgbd_camera_offset_x" value="-0.29545"/>
+   <xacro:property name="rear_rgbd_camera_offset_y" value="0.0"/>
+   <xacro:property name="rear_rgbd_camera_offset_z" value="0.1662"/>
+   <xacro:property name="gps_offset_x" value="-0.365"/>
+   <xacro:property name="gps_offset_y" value="-0.167"/>
+   <xacro:property name="gps_offset_z" value="0.302"/>
+  <xacro:macro name="rb_theron" params="prefix publish_bf hq load_kinematics_file gpu:=false">
+    <!-- *************** -->
+    <!-- Robots Elements -->
+    <!-- *************** -->
+    <!-- Here we create the robot elements using the xacro:macros imported at the beggining of this file -->
+ 	<!-- rb_theron_omni base -->
+   <xacro:rb_theron_omni_base prefix="$(arg prefix)" publish_bf="true" hq="${hq}" />
+   <xacro:omni_wheel prefix="$(arg prefix)front_right" parent="$(arg prefix)base_link" reflect="false" hq="${hq}">
+     <origin xyz="${wheel_offset_x} -${wheel_offset_y} ${wheel_offset_z}" rpy="0 0 0"/>
+   </xacro:omni_wheel>
+   <xacro:omni_wheel prefix="$(arg prefix)front_left" parent="$(arg prefix)base_link" reflect="true" hq="${hq}">
+     <origin xyz="${wheel_offset_x} ${wheel_offset_y} ${wheel_offset_z}" rpy="0 0 0"/>
+   </xacro:omni_wheel>
+   <xacro:omni_wheel prefix="$(arg prefix)back_left" parent="$(arg prefix)base_link" reflect="true" hq="${hq}">
+     <origin xyz="-${wheel_offset_x} ${wheel_offset_y} ${wheel_offset_z}" rpy="0 0 0"/>
+   </xacro:omni_wheel>
+   <xacro:omni_wheel prefix="$(arg prefix)back_right" parent="$(arg prefix)base_link" reflect="false" hq="${hq}">
+     <origin xyz="-${wheel_offset_x} -${wheel_offset_y} ${wheel_offset_z}" rpy="0 0 0"/>
+   </xacro:omni_wheel>
+       <!-- IMU -->
+   <xacro:sensor_imu_hector prefix="$(arg prefix)imu" parent="$(arg prefix)base_link">
+     <origin xyz="${imu_offset_x} ${imu_offset_y} ${imu_offset_z}" rpy="0 0 0"/>
+   </xacro:sensor_imu_hector>
+   <!-- SENSORS -->
+   <xacro:sensor_sick_nanoscan3 prefix="$(arg prefix)front_laser" parent="$(arg prefix)base_link" prefix_topic="front_laser" gpu="${gpu}">
+     <origin xyz="${front_laser_offset_x} ${front_laser_offset_y} ${front_laser_offset_z}" rpy="0 ${-PI} ${3/4*PI}" />
+   </xacro:sensor_sick_nanoscan3>
+   <xacro:sensor_sick_nanoscan3 prefix="$(arg prefix)rear_laser" parent="$(arg prefix)base_link" prefix_topic="rear_laser" gpu="${gpu}">
+     <origin xyz="${rear_laser_offset_x} ${rear_laser_offset_y} ${rear_laser_offset_z}" rpy="0 ${-PI} ${-1/4*PI}" />
+   </xacro:sensor_sick_nanoscan3>
+   <xacro:sensor_intel_d435 prefix="$(arg prefix)front_rgbd_camera" parent="$(arg prefix)base_link" prefix_topic="front_rgbd_camera">
+     <origin xyz="${front_rgbd_camera_offset_x} ${front_rgbd_camera_offset_y} ${front_rgbd_camera_offset_z}" rpy="0 0 0"/>
+   </xacro:sensor_intel_d435>
+   <xacro:sensor_intel_d435 prefix="$(arg prefix)rear_rgbd_camera" parent="$(arg prefix)base_link" prefix_topic="rear_rgbd_camera">
+   <origin xyz="${rear_rgbd_camera_offset_x} ${rear_rgbd_camera_offset_y} ${rear_rgbd_camera_offset_z}" rpy="0 ${-PI} 0"/>
+ </xacro:sensor_intel_d435>
+  </xacro:macro>
+  <!-- Gazebo ros control pluggins -->
+  <xacro:ros_control/>
+  <xacro:if value="$(arg ros_planar_move_plugin)">
+    <xacro:omni_steering prefix="$(arg prefix)" publish_tf="true"/>
+  </xacro:if>
+  <xacro:rb_theron prefix="$(arg prefix)" publish_bf="true" hq="true" load_kinematics_file="$(arg load_kinematics_file)" gpu="$(arg use_gpu_for_simulation)"/>
 </robot>

File: rb_theron_description/urdf/wheels/omni_wheel.urdf.xacro (robot description, xacro)
@@ -1,141 +1,79 @@
 <?xml version="1.0"?>
-<robot name="omni" xmlns:xacro="http://www.ros.org/wiki/xacro">
+<robot name="wheel" xmlns:xacro="http://wiki.ros.org/xacro">
   <xacro:property name="M_PI" value="3.1415926535897931" />
-  <!-- omni support parameters -->
-  <xacro:property name="omni_support_mass" value="1.5" /> <!-- in kg-->
-  <!-- omni wheel parameters -->
-  <xacro:property name="wheel_radius" value="0.050" />
-  <xacro:property name="omni_height" value="0.025" />
-  <xacro:property name="omni_mass" value="0.25" /> <!-- in kg-->
-  <!-- omni wheel offset-->
-  <xacro:property name="omni_wheel_offset_x" value="-0.033" />
-  <!-- x,y,z in translation from omni_support to the center of the omni wheel-->
-  <xacro:property name="omni_wheel_offset_y" value="0.0" />
-  <xacro:property name="omni_wheel_offset_z" value="-0.071" />
+  <!-- Wheels -->
+  <xacro:property name="omni_wheel_radius" value="0.0762" />
+  <xacro:property name="omni_wheel_height" value="0.087" />
+  <xacro:property name="omni_wheel_mass" value="6.5" /> <!-- in kg-->
   <xacro:macro name="cylinder_inertia" params="m r h">
     <inertia  ixx="${m*(3*r*r+h*h)/12}" ixy = "0" ixz = "0"
-              iyy="${m*(3*r*r+h*h)/12}" iyz = "0"
-              izz="${m*r*r/2}" />
+              iyy="${m*r*r/2}" iyz = "0"
+              izz="${m*(3*r*r+h*h)/12}" />
   </xacro:macro>
-  <xacro:macro name="omni" params="prefix parent *origin hq">
-  <!--omni SUPPORT -->
-  <joint name="${prefix}_joint_support" type="continuous">
+  <xacro:macro name="omni_wheel" params="prefix parent *origin reflect hq">
+    <joint name="${prefix}_wheel_joint" type="continuous">
       <parent link="${parent}"/>
-      <child link="${prefix}_support"/>
+      <child link="${prefix}_wheel_link"/>
       <xacro:insert_block name="origin" />
-      <axis xyz="0 0 1" rpy="0 ${M_PI} 0" />
+      <axis xyz="0 1 0" rpy="0 0 0" />
       <limit effort="100" velocity="100"/>
-      <!-- joint_properties damping="1.5" friction="1.5"/ -->
-      <dynamics damping="0" friction="0.01"/>
+      <joint_properties damping="0.0" friction="0.0"/>
     </joint>
-    <link name="${prefix}_support">
+    <link name="${prefix}_wheel_link">
       <visual>
-        <origin xyz="0 0 0" rpy="0 0 0" />
+        <xacro:if value="${hq}">
+          <origin xyz="0 0 0" rpy="0 0 0" />
+          <xacro:if value="${reflect}">
+            <geometry>
+              <mesh filename="package://rb_theron_description/meshes/wheels/omni_wheel.stl" />
+            </geometry>
+          </xacro:if>
+          <xacro:unless value="${reflect}">
+            <geometry>
+              <mesh filename="package://rb_theron_description/meshes/wheels/omni_wheel.stl" />
+            </geometry>
+		  </xacro:unless>
+        </xacro:if>
+        <xacro:unless value="${hq}">
+          <origin xyz="0 0 0" rpy="0 0 0" />
           <geometry>
-	       <mesh filename="package://rb_theron_description/meshes/wheels/omni_wheel.stl" />
+            <sphere radius="${omni_wheel_radius}" />
           </geometry>
+        </xacro:unless>
+        <material name="darkgrey">
+           <color rgba="0.2 0.2 0.2 1"/>
+        </material>
       </visual>
       <collision>
-        <origin xyz="0 0 0" rpy="0 0 0" />
-          <geometry>
-	       <mesh filename="package://rb_theron_description/meshes/wheels/omni_wheel.dae" />
-          </geometry>
+				<origin xyz="0 0 0" rpy="${PI/2} 0 0" />
+        <geometry>
+          <!--sphere radius="${omni_wheel_radius}" /-->
+					<cylinder length="${omni_wheel_height}" radius="${omni_wheel_radius}" />
+					<!-- sphere radius="${omni_wheel_radius}"/-->
+        </geometry>
       </collision>
       <inertial>
-        <mass value="${omni_support_mass}" />
+        <mass value="${omni_wheel_mass}" />
         <origin xyz="0 0 0" />
-        <xacro:cylinder_inertia  m="${omni_support_mass}" r="0.010" h="0.010" />  <!--Check these values -->
+        <xacro:cylinder_inertia  m="${omni_wheel_mass}" r="${omni_wheel_radius}" h="${omni_wheel_height}" />
       </inertial>
     </link>
-  <!--omni WHEEL -->
-  <!-- xacro:omni_wheel prefix="${prefix}" parent="${prefix}_support" hq="${hq}" -->
-  <xacro:omni_wheel prefix="${prefix}" parent="${prefix}_support" hq="${hq}">
-		<origin xyz="${omni_wheel_offset_x} ${omni_wheel_offset_y} ${omni_wheel_offset_z}" rpy="0 0 0"/>
-   </xacro:omni_wheel>
- </xacro:macro>
- <xacro:macro name="omni_wheel" params="prefix parent *origin hq">
-     <joint name="${prefix}joint_wheel" type="continuous">
-       <parent link="${parent}"/>
-       <child link="${prefix}_wheel"/>
-       <insert_block name="origin" />
-       <axis xyz="0 1 0" rpy="0 0 0" />
-       <limit effort="100" velocity="100"/>
-       <joint_properties damping="0.1" friction="0.1"/>
-    </joint>
-    <link name="${prefix}_wheel">
-      <visual>
-        <!-- HIGH RESOLUTION WHEELS -->
-     <!-- xacro:if value="${hq}">
-          <origin xyz="0 0 0" rpy="0 0 0" />
-          <geometry>
-		<mesh filename="package://rb_theron_description/meshes/wheels/mcq_prototype_omni_wheel.dae" />
-          </geometry>
-        </xacro:if -->
-       <!-- LOW RESOLUTION WHEELS -->
-       <!-- xacro:unless value="${hq}" -->
-          <origin xyz="0 0 0" rpy="0 0 0" />
-          <geometry>
-            <cylinder length="${omni_height}" radius="${wheel_radius}" />
-            <!-- sphere radius="${wheel_radius}"/ -->
-          </geometry>
-        <!-- /xacro:unless -->
-      </visual>
-     <collision>
-	  <origin xyz="0 0 0" rpy="${M_PI/2} 0 0" />
-	  <!-- origin xyz="0 0 0" rpy="0 0 0" / -->
-        <geometry>
-		  <!-- mesh filename="package://rb_theron_description/meshes/wheels/mcq_prototype_omni_wheel.dae" / -->
-          <cylinder length="${omni_height}" radius="${wheel_radius}" />
-          <!-- sphere radius="${wheel_radius}"/ -->
-        </geometry>
-		<surface>
-          <bounce restitution_coefficient = "1"/>
-		</surface>
-      </collision>
-      <inertial>
-        <mass value="${omni_mass}" />
-        <origin xyz="0 0 0" />
-        <xacro:cylinder_inertia  m="${omni_mass}" r="${wheel_radius}" h="${omni_height}" />
-      </inertial>
-    </link>
-  <!-- Transmission is important to link the joints and the controller -->
-    <transmission name="${prefix}_support_joint_trans">
+    <transmission name="${prefix}_wheel_joint_trans">
       <type>transmission_interface/SimpleTransmission</type>
-      <joint name="${prefix}_joint_support">
-          <hardwareInterface>hardware_interface/EffortJointInterface</hardwareInterface>
+      <joint name="${prefix}_wheel_joint" >
+        <hardwareInterface>hardware_interface/VelocityJointInterface</hardwareInterface>
       </joint>
-      <actuator name="${prefix}_support_joint_motor">
-        <mechanicalReduction>1</mechanicalReduction>
-      	<motorTorqueConstant>1</motorTorqueConstant>
+      <actuator name="${prefix}_wheel_joint_motor">
+         <mechanicalReduction>1</mechanicalReduction>
       </actuator>
     </transmission>
-    <transmission name="${prefix}_wheel_joint_trans">
-      <type>transmission_interface/SimpleTransmission</type>
-      <joint name="${prefix}joint_wheel">
-          <hardwareInterface>hardware_interface/EffortJointInterface</hardwareInterface>
-      </joint>
-      <actuator name="${prefix}_wheel_joint_motor">
-        <mechanicalReduction>1</mechanicalReduction>
-		<motorTorqueConstant>1</motorTorqueConstant>
-      </actuator>
-    </transmission>
-    <gazebo reference="${prefix}_support">
-			<mu1 value="5.0"/>
-			<mu2 value="0.5"/>
-			<kp value="10000000.0" />
-			<kd value="1.0" />
-			<fdir1 value="1 0 0"/>
-      <turnGravityOff>false</turnGravityOff>
+    <gazebo reference="${prefix}_wheel_link">
+		<mu1 value="0.0"/>
+		<mu2 value="0.0"/>
+		<kp value="10000000.0" />
+		<kd value="1.0" />
+		<fdir1 value="1 0 0"/>
+        <turnGravityOff>false</turnGravityOff>
     </gazebo>
-     <gazebo reference="${prefix}_wheel">
-			<mu1 value="100.0"/>
-			<mu2 value="100.0"/>
-			<!-- kp value="10000000.0" / -->
-			<kp value="100000.0" />
-			<kd value="100.0" />
-			<!-- fdir1 value="1 0 0"/ -->
-			<material>Gazebo/Black</material>
-			<turnGravityOff>false</turnGravityOff>
-    </gazebo>
- </xacro:macro>
+  </xacro:macro>
 </robot>

Commit message: Update rb_theron_omni urdf to delete unnecesary logos

File: rb_theron_description/robots/rb_theron_omni.urdf.xacro (robot description, xacro)
@@ -14,5 +14,5 @@
   <xacro:property name="hq" value="true" />
   <xacro:arg name="prefix" default="robot_"/>
-  <xacro:arg name="ros_planar_move_plugin" default="false"/>
+  <xacro:arg name="ros_planar_move_plugin" default="true"/>
   <xacro:arg name="load_kinematics_file" default="false"/> <!-- Necesarry for ur_description compatible with official ur drivers-->
   <xacro:arg name="use_gpu_for_simulation" default="false"/>

File: rb_theron_description/urdf/bases/rb_theron_omni_base.urdf.xacro (robot description, xacro)
@@ -72,5 +72,5 @@
     <child link="${prefix}base_chapa" />
   </joint-->
-  <!-- LOGO ROBOTNIK IZQUIERDO -->
+  <!-- LOGO ROBOTNIK IZQUIERDO >
   <link name="${prefix}base_logo_left">
   <visual>
@@ -88,6 +88,6 @@
     <parent link="${prefix}base_link"/>
     <child link="${prefix}base_logo_left" />
-  </joint>
-  <!-- LOGO ROBOTNIK DERECHO -->
+  </joint-->
+  <!-- LOGO ROBOTNIK DERECHO >
   <link name="${prefix}base_logo_right">
   <visual>
@@ -105,6 +105,6 @@
     <parent link="${prefix}base_link"/>
     <child link="${prefix}base_logo_right" />
-  </joint>
-  <!-- LOGO ROBOTNIK FRONTAL -->
+  </joint-->
+  <!-- LOGO ROBOTNIK FRONTAL >
   <link name="${prefix}base_logo_front">
   <visual>
@@ -122,6 +122,6 @@
     <parent link="${prefix}base_link"/>
     <child link="${prefix}base_logo_front" />
-  </joint>
-  <!-- LOGO ROBOTNIK TRASERO -->
+  </joint-->
+  <!-- LOGO ROBOTNIK TRASERO >
   <link name="${prefix}base_logo_rear">
   <visual>
@@ -139,5 +139,5 @@
     <parent link="${prefix}base_link"/>
     <child link="${prefix}base_logo_rear" />
-  </joint>
+  </joint-->
    <!-- DOCKING CONTACT -->
     <link name="${prefix}base_docking_contact">
