Commit message: description/robots: Update caster positions in rb_theron_base.urdf.xacro

File: rb_theron_description/robots/rb_theron_base.urdf.xacro (robot description, xacro)
@@ -9,5 +9,5 @@
 	<xacro:include filename="$(find rb_theron_description)/urdf/bases/theron_base.urdf.xacro" />
 	<!-- Import wheels -->
-	<xacro:include filename="$(find rb_theron_description)/urdf/wheels/rubber_wheel_150.urdf.xacro" />
+	<xacro:include filename="$(find rb_theron_description)/urdf/wheels/rubber_wheel_140.urdf.xacro" />
 	<!-- Import casters -->
 	<xacro:include filename="$(find rb_theron_description)/urdf/wheels/castor.urdf.xacro" />
@@ -36,16 +36,18 @@
   		<origin xyz="${wheel_offset_x} ${wheel_offset_y} ${wheel_offset_z}" rpy="0 0 0"/>
   	</xacro:rubber_wheel>
+<!-- To do: fix castor wheels
   	<xacro:caster prefix="${prefix}front_left" parent="${prefix}base_link" hq="${hq}">
-  		<origin xyz="0.235 0.1825 0.046" rpy="0 0 0"/>
+  		<origin xyz="0.235 0.1825 0.0448" rpy="0 0 0"/>
   	</xacro:caster>
   	<xacro:caster prefix="${prefix}front_right" parent="${prefix}base_link" hq="${hq}">
-  		<origin xyz="0.235 -0.1825 0.046" rpy="0 0 0"/>
+  		<origin xyz="0.235 -0.1825 0.0448" rpy="0 0 0"/>
   	</xacro:caster>
   	<xacro:caster prefix="${prefix}rear_left" parent="${prefix}base_link" hq="${hq}">
-  		<origin xyz="-0.235 0.1825 0.046" rpy="0 0 0"/>
+  		<origin xyz="-0.235 0.1825 0.0448" rpy="0 0 0"/>
   	</xacro:caster>
   	<xacro:caster prefix="${prefix}rear_right" parent="${prefix}base_link" hq="${hq}">
-  		<origin xyz="-0.235 -0.1825 0.046" rpy="0 0 0"/>
+  		<origin xyz="-0.235 -0.1825 0.0448" rpy="0 0 0"/>
   	</xacro:caster>
+-->
   </xacro:macro>
 </robot>

Commit message: Correct castor wheel for simulation in Noetic

File: rb_theron_description/robots/rb_theron_base.urdf.xacro (robot description, xacro)
@@ -36,5 +36,5 @@
   		<origin xyz="${wheel_offset_x} ${wheel_offset_y} ${wheel_offset_z}" rpy="0 0 0"/>
   	</xacro:rubber_wheel>
-<!-- To do: fix castor wheels
+<!-- Castor wheels-->
   	<xacro:caster prefix="${prefix}front_left" parent="${prefix}base_link" hq="${hq}">
   		<origin xyz="0.235 0.1825 0.0448" rpy="0 0 0"/>
@@ -49,5 +49,4 @@
   		<origin xyz="-0.235 -0.1825 0.0448" rpy="0 0 0"/>
   	</xacro:caster>
--->
   </xacro:macro>
 </robot>

File: rb_theron_description/urdf/wheels/castor.urdf.xacro (robot description, xacro)
@@ -22,6 +22,6 @@
   <joint name="${prefix}joint_support" type="continuous">
       <parent link="${parent}"/>
-      <child link="${prefix}support"/>
-      <insert_block name="origin" />
+      <child link="${prefix}_support"/>
+      <xacro:insert_block name="origin" />
       <axis xyz="0 0 1" rpy="0 ${M_PI} 0" />
       <limit effort="100" velocity="100"/>
@@ -29,5 +29,5 @@
       <dynamics damping="0" friction="0.01"/>
     </joint>
-    <link name="${prefix}support">
+    <link name="${prefix}_support">
       <visual>
         <origin xyz="0 0 0" rpy="0 0 0" />
@@ -36,10 +36,10 @@
           </geometry>
       </visual>
-      <!--collision>
+      <collision>
         <origin xyz="0 0 0" rpy="0 0 0" />
           <geometry>
 	       <mesh filename="package://rb_theron_description/meshes/wheels/castor_wheel.dae" />
           </geometry>
-      </collision-->
+      </collision>
       <inertial>
         <mass value="${caster_support_mass}" />
@@ -49,6 +49,6 @@
     </link>
   <!--CASTER WHEEL -->
-  <!-- xacro:caster_wheel prefix="${prefix}" parent="${prefix}support" hq="${hq}" -->
-  <xacro:caster_wheel prefix="${prefix}" parent="${prefix}support" hq="${hq}">
+  <!-- xacro:caster_wheel prefix="${prefix}" parent="${prefix}_support" hq="${hq}" -->
+  <xacro:caster_wheel prefix="${prefix}" parent="${prefix}_support" hq="${hq}">
 		<origin xyz="${caster_wheel_offset_x} ${caster_wheel_offset_y} ${caster_wheel_offset_z}" rpy="0 0 0"/>
    </xacro:caster_wheel>
@@ -57,5 +57,5 @@
      <joint name="${prefix}joint_wheel" type="continuous">
        <parent link="${parent}"/>
-       <child link="${prefix}wheel"/>
+       <child link="${prefix}_wheel"/>
        <insert_block name="origin" />
        <axis xyz="0 1 0" rpy="0 0 0" />
@@ -63,5 +63,5 @@
        <joint_properties damping="0.1" friction="0.1"/>
     </joint>
-    <link name="${prefix}wheel">
+    <link name="${prefix}_wheel">
       <visual>
         <!-- HIGH RESOLUTION WHEELS -->
@@ -74,5 +74,5 @@
        <!-- LOW RESOLUTION WHEELS -->
        <!-- xacro:unless value="${hq}" -->
-          <origin xyz="0 0 0" rpy="${M_PI/2} 0 0" />
+          <origin xyz="0 0 0" rpy="0 0 0" />
           <geometry>
             <cylinder length="${caster_height}" radius="${caster_radius}" />
@@ -100,25 +100,25 @@
     </link>
   <!-- Transmission is important to link the joints and the controller -->
-    <transmission name="${prefix}support_joint_trans">
+    <transmission name="${prefix}_support_joint_trans">
       <type>transmission_interface/SimpleTransmission</type>
       <joint name="${prefix}joint_support">
           <hardwareInterface>hardware_interface/EffortJointInterface</hardwareInterface>
       </joint>
-      <actuator name="${prefix}support_joint_motor">
+      <actuator name="${prefix}_support_joint_motor">
         <mechanicalReduction>1</mechanicalReduction>
       	<motorTorqueConstant>1</motorTorqueConstant>
       </actuator>
     </transmission>
-    <transmission name="${prefix}wheel_joint_trans">
+    <transmission name="${prefix}_wheel_joint_trans">
       <type>transmission_interface/SimpleTransmission</type>
       <joint name="${prefix}joint_wheel">
           <hardwareInterface>hardware_interface/EffortJointInterface</hardwareInterface>
       </joint>
-      <actuator name="${prefix}wheel_joint_motor">
+      <actuator name="${prefix}_wheel_joint_motor">
         <mechanicalReduction>1</mechanicalReduction>
 		<motorTorqueConstant>1</motorTorqueConstant>
       </actuator>
     </transmission>
-    <!-- gazebo reference="${prefix}support">
+    <gazebo reference="${prefix}_support">
 			<mu1 value="5.0"/>
 			<mu2 value="0.5"/>
@@ -127,5 +127,5 @@
 			<fdir1 value="1 0 0"/>
       <turnGravityOff>false</turnGravityOff>
-    </gazebo -->
+    </gazebo>
      <gazebo reference="${prefix}_wheel">
 			<mu1 value="100.0"/>

Commit message: Use v4 theron base as standard

File: rb_theron_description/robots/rb_theron_base.urdf.xacro (robot description, xacro)
@@ -7,5 +7,5 @@
 	<!-- First we import all posible elements defined in the urdf.xacro files. All these elements are defined as macro:xacros -->
 	<!-- Import differential base elements -->
-	<xacro:include filename="$(find rb_theron_description)/urdf/bases/theron_base.urdf.xacro" />
+	<xacro:include filename="$(find rb_theron_description)/urdf/bases/rb_theron_base_v4.urdf.xacro" />
 	<!-- Import wheels -->
 	<xacro:include filename="$(find rb_theron_description)/urdf/wheels/rubber_wheel_150.urdf.xacro" />
@@ -26,6 +26,6 @@
 	<!-- *************** -->
   <xacro:macro name="rb_theron_base" params="prefix hq use_sim">
-    <!-- rbogie base -->
-  	<xacro:theron_base prefix="${prefix}" publish_bf="true" hq="${hq}" />
+    <!-- rb_theron base -->
+  	<xacro:rb_theron_base_v4 prefix="${prefix}" publish_bf="true" hq="${hq}" />
     <xacro:gazebo_colors prefix="${prefix}"/>
   	<!-- WHEELS -->

File: rb_theron_description/robots/rb_theron_omni.urdf.xacro (robot description, xacro)
@@ -5,6 +5,6 @@
   <!-- ***************** -->
   <!-- First we import all posible elements defined in the urdf.xacro files. All these elements are defined as macro:xacros -->
-  <!-- Import rb_theron_omni base elements -->
-  <xacro:include filename="$(find rb_theron_description)/urdf/bases/rb_theron_omni_base.urdf.xacro" />
+  <!-- Import rb_theron_v4 base elements -->
+  <xacro:include filename="$(find rb_theron_description)/urdf/bases/rb_theron_base_v4.urdf.xacro" />
   <!-- Import rb_theron_omni wheels -->
   <xacro:include filename="$(find rb_theron_description)/urdf/wheels/omni_wheel.urdf.xacro" />
@@ -51,6 +51,6 @@
     <!-- *************** -->
     <!-- Here we create the robot elements using the xacro:macros imported at the beggining of this file -->
- 	<!-- rb_theron_omni base -->
-   <xacro:rb_theron_omni_base prefix="$(arg prefix)" publish_bf="true" hq="${hq}" />
+ 	<!-- rb_theron_v4 base -->
+   <xacro:rb_theron_base_v4 prefix="$(arg prefix)" publish_bf="true" hq="${hq}" />
    <xacro:omni_wheel prefix="$(arg prefix)front_right" parent="$(arg prefix)base_link" reflect="false" hq="${hq}">
      <origin xyz="${wheel_offset_x} -${wheel_offset_y} ${wheel_offset_z}" rpy="0 0 0"/>

File: rb_theron_description/urdf/bases/rb_theron_base_v4.urdf.xacro (robot description, xacro)
@@ -1,6 +1,6 @@
 <?xml version="1.0"?>
-<robot name="rb_theron_omni" xmlns:xacro="http://wiki.ros.org/xacro">
+<robot name="rb_theron_v4" xmlns:xacro="http://wiki.ros.org/xacro">
   <xacro:include filename="$(find rb_theron_description)/urdf/bases/base.gazebo.xacro" />
-  <xacro:macro name="rb_theron_v4_base" params="prefix publish_bf hq">
+  <xacro:macro name="rb_theron_base_v4" params="prefix publish_bf hq">
   <!-- Robot mechanical and motor parameters -->
   <xacro:property name="PI" value="3.1415926535897931"/>
