Commit message: Update 2d files

File: rb_theron_description/robots/rb_theron.urdf.xacro (robot description, xacro)
@@ -13,5 +13,5 @@
 	<xacro:include filename="$(find rb_theron_description)/urdf/wheels/castor.urdf.xacro" />
 	<!-- Import rocker bogie -->
-	<xacro:include filename="$(find rb_theron_description)/urdf/rocker/mcq_prototype_rocker.urdf.xacro" />
+	<xacro:include filename="$(find rb_theron_description)/urdf/rocker/rb_theron_rocker.urdf.xacro" />
 	<!-- Import all available sensors -->
 	<xacro:include filename="$(find robotnik_sensors)/urdf/all_sensors.urdf.xacro" />

File: rb_theron_description/urdf/bases/theron_base.urdf.xacro (robot description, xacro)
@@ -69,5 +69,5 @@
         <xacro:if value="${hq}">
           <geometry>
-            <mesh filename="package://rb_theron_description/meshes/bases/mcq_prototype_bottom_cover.dae"/>
+            <mesh filename="package://rb_theron_description/meshes/bases/rb_theron_bottom_cover.dae"/>
           </geometry>
         </xacro:if>
@@ -84,5 +84,5 @@
         <origin xyz="0 0 0" rpy="0 0 0 " />
         <geometry>
-          <mesh filename="package://rb_theron_description/meshes/bases/mcq_prototype_bottom_cover.dae"/>
+          <mesh filename="package://rb_theron_description/meshes/bases/rb_theron_bottom_cover.dae"/>
         </geometry>
       </collision>

File: rb_theron_description/urdf/rocker/rb_theron_rocker.urdf.xacro (robot description, xacro)
@@ -36,10 +36,10 @@
           <xacro:if value="${reflect}">
             <geometry>
-	          <mesh filename="package://rb_theron_description/meshes/rocker/mcq_prototype_rocker_r.dae" />
+	          <mesh filename="package://rb_theron_description/meshes/rocker/rb_theron_rocker_r.dae" />
             </geometry>
           </xacro:if>
           <xacro:unless value="${reflect}">
             <geometry>
-              <mesh filename="package://rb_theron_description/meshes/rocker/mcq_prototype_rocker_l.dae" />
+              <mesh filename="package://rb_theron_description/meshes/rocker/rb_theron_rocker_l.dae" />
             </geometry>
 		  </xacro:unless>
@@ -49,10 +49,10 @@
           <xacro:if value="${reflect}">
             <geometry>
-	          <mesh filename="package://rb_theron_description/meshes/rocker/mcq_prototype_rocker_r.dae" />
+	          <mesh filename="package://rb_theron_description/meshes/rocker/rb_theron_rocker_r.dae" />
             </geometry>
           </xacro:if>
           <xacro:unless value="${reflect}">
             <geometry>
-              <mesh filename="package://rb_theron_description/meshes/rocker/mcq_prototype_rocker_l.dae" />
+              <mesh filename="package://rb_theron_description/meshes/rocker/rb_theron_rocker_l.dae" />
             </geometry>
 		  </xacro:unless>

File: rb_theron_description/urdf/wheels/castor.urdf.xacro (robot description, xacro)
@@ -33,5 +33,5 @@
         <origin xyz="0 0 0" rpy="0 0 0" />
           <geometry>
-	       <mesh filename="package://rb_theron_description/meshes/wheels/mcq_prototype_base_castor.dae" />
+	       <mesh filename="package://rb_theron_description/meshes/wheels/rb_theron_base_castor.dae" />
           </geometry>
       </visual>
@@ -39,5 +39,5 @@
         <origin xyz="0 0 0" rpy="0 0 0" />
           <geometry>
-	       <mesh filename="package://rb_theron_description/meshes/wheels/mcq_prototype_base_castor.dae" />
+	       <mesh filename="package://rb_theron_description/meshes/wheels/rb_theron_base_castor.dae" />
           </geometry>
       </collision>
@@ -69,5 +69,5 @@
           <origin xyz="0 0 0" rpy="0 0 0" />
           <geometry>
-		<mesh filename="package://rb_theron_description/meshes/wheels/mcq_prototype_castor_wheel.dae" />
+		<mesh filename="package://rb_theron_description/meshes/wheels/rb_theron_castor_wheel.dae" />
           </geometry>
         </xacro:if -->
@@ -85,5 +85,5 @@
 	  <!-- origin xyz="0 0 0" rpy="0 0 0" / -->
         <geometry>
-		  <!-- mesh filename="package://rb_theron_description/meshes/wheels/mcq_prototype_castor_wheel.dae" / -->
+		  <!-- mesh filename="package://rb_theron_description/meshes/wheels/rb_theron_castor_wheel.dae" / -->
           <cylinder length="${caster_height}" radius="${caster_radius}" />
           <!-- sphere radius="${caster_radius}"/ -->

Commit message: Updates robot description to visualize wheels

File: rb_theron_description/robots/rb_theron.urdf.xacro (robot description, xacro)
@@ -23,13 +23,7 @@
 	<xacro:property name="PI" value="3.1415926535897931"/>
 	<!-- Wheel parameters -->
-	<!-- x,y,z in translation from base_link to the center of the wheel -->
-	<xacro:property name="rocker_offset_x" value="0.1175" />
-	<xacro:property name="rocker_offset_y" value="0.1725" />
-	<xacro:property name="rocker_offset_z" value="0.0428" />
-	<!-- Castor paramters -->
-	<xacro:property name="caster_offset_x" value="-0.235" />
-	<xacro:property name="caster_offset_y" value="0.1725" />
-	<xacro:property name="caster_offset_z" value="0.0428" />
-	<xacro:property name="wheel_offset_z" value="0.015" />
+	<xacro:property name="wheel_offset_x" value="0" />
+	<xacro:property name="wheel_offset_y" value="0.2545" />
+	<xacro:property name="wheel_offset_z" value="0.0428" />
 	<!-- Flag to select the high or low quality model -->
 	<xacro:property name="hq" value="true" />
@@ -46,16 +40,10 @@
 	<xacro:gazebo_colors prefix="$(arg prefix)"/>
 	<!-- WHEELS -->
-	<xacro:rocker prefix="$(arg prefix)right" parent="$(arg prefix)base_link" reflect="true" hq="${hq}">
-		<origin xyz="${rocker_offset_x} -${rocker_offset_y} ${rocker_offset_z}" rpy="0 0 0"/>
-	</xacro:rocker>
-	<xacro:rocker prefix="$(arg prefix)left" parent="$(arg prefix)base_link" reflect="false" hq="${hq}">
-		<origin xyz="${rocker_offset_x} ${rocker_offset_y} ${rocker_offset_z}" rpy="0 0 0"/>
-	</xacro:rocker>
-	<xacro:caster prefix="$(arg prefix)left" parent="$(arg prefix)base_link" hq="${hq}">
-		<origin xyz="${caster_offset_x} ${caster_offset_y} ${caster_offset_z}" rpy="0 0 0"/>
-	</xacro:caster>
-	<xacro:caster prefix="$(arg prefix)right" parent="$(arg prefix)base_link" hq="${hq}">
-		<origin xyz="${caster_offset_x} ${-caster_offset_y} ${caster_offset_z}" rpy="0 0 0"/>
-	</xacro:caster>
+	<xacro:rubber_wheel prefix="$(arg prefix)right" parent="$(arg prefix)base_link" hq="${hq}">
+		<origin xyz="${wheel_offset_x} ${-wheel_offset_y} ${wheel_offset_z}" rpy="0 0 0"/>
+	</xacro:rubber_wheel>
+	<xacro:rubber_wheel prefix="$(arg prefix)left" parent="$(arg prefix)base_link" hq="${hq}">
+		<origin xyz="${wheel_offset_x} ${wheel_offset_y} ${wheel_offset_z}" rpy="0 0 0"/>
+	</xacro:rubber_wheel>
 	<!-- SENSORS -->
 	<!-- TODO: Should be intel_t265 -->

Commit message: description: update model (clean & fix) and remove unused files

File: rb_theron_description/robots/rb_theron.urdf.xacro (robot description, xacro)
@@ -24,6 +24,6 @@
 	<!-- Wheel parameters -->
 	<xacro:property name="wheel_offset_x" value="0" />
-	<xacro:property name="wheel_offset_y" value="0.2545" />
-	<xacro:property name="wheel_offset_z" value="0.0428" />
+	<xacro:property name="wheel_offset_y" value="0.2516" />
+	<xacro:property name="wheel_offset_z" value="0.0" />
 	<!-- Flag to select the high or low quality model -->
 	<xacro:property name="hq" value="true" />
@@ -46,10 +46,16 @@
 		<origin xyz="${wheel_offset_x} ${wheel_offset_y} ${wheel_offset_z}" rpy="0 0 0"/>
 	</xacro:rubber_wheel>
-	<!-- SENSORS -->
-	<!-- TODO: Should be intel_t265 -->
-	<!-- TODO: Moved 0.01 in x, otherwise the camera is still inside the robot -->
-	<xacro:sensor_r430 prefix="$(arg prefix)front_realsense_camera" parent="$(arg prefix)base_link" prefix_topic="front_realsense_camera">
-		<origin xyz="0.3305 0.0 0.1468" rpy="0 0 0"/>
-	</xacro:sensor_r430>
+	<xacro:caster prefix="$(arg prefix)front_left" parent="$(arg prefix)base_link" hq="${hq}">
+		<origin xyz="0.235 0.1825 0.046" rpy="0 0 0"/>
+	</xacro:caster>
+	<xacro:caster prefix="$(arg prefix)front_right" parent="$(arg prefix)base_link" hq="${hq}">
+		<origin xyz="0.235 -0.1825 0.046" rpy="0 0 0"/>
+	</xacro:caster>
+	<xacro:caster prefix="$(arg prefix)rear_left" parent="$(arg prefix)base_link" hq="${hq}">
+		<origin xyz="-0.235 0.1825 0.046" rpy="0 0 0"/>
+	</xacro:caster>
+	<xacro:caster prefix="$(arg prefix)rear_right" parent="$(arg prefix)base_link" hq="${hq}">
+		<origin xyz="-0.235 -0.1825 0.046" rpy="0 0 0"/>
+	</xacro:caster>
   <!-- TODO: Moved 0.01 in x, otherwise the camera is still inside the robot -->
 	<xacro:sensor_orbbec_astra prefix="$(arg prefix)front_rgbd_camera" parent="$(arg prefix)base_link" prefix_topic="front_rgbd_camera">

File: rb_theron_description/urdf/bases/theron_base.urdf.xacro (robot description, xacro)
@@ -30,8 +30,8 @@
     <link name="${prefix}base_link">
       <inertial>
-        <mass value="50.0" />
-        <origin xyz="-0.120 0 0" />
-	    <xacro:box_inertia_robot m="50" x="0.700" y="0.600" z="0.350"/>
-      </inertial>
+      <mass value="45" />
+      <origin xyz="0.0 0.0 0.0" />
+      <xacro:solid_cuboid_inertia m="45" w="0.3275" h="0.2775" d="0.1525" />
+     </inertial>
       <visual>
         <origin xyz="0 0 0" rpy="0 0 0" />
@@ -52,53 +52,11 @@
       </visual>
       <collision>
-        <origin xyz="0 0 0" rpy="0 0 0 " />
+        <origin xyz="0 0 0.005" rpy="0 0 0 " />
         <geometry>
-          <!--box size="0.390 0.240 0.165"/-->
-          <mesh filename="package://rb_theron_description/meshes/bases/theron_base.stl"/>
+          <!--box size="0.05 0.05 0.01"/-->
+          <mesh filename="package://rb_theron_description/meshes/bases/theron_base.dae"/>
         </geometry>
       </collision>
     </link>
-    <!-- <link name="${prefix}bottom_cover_link">
-      <inertial>
-        <mass value="2.0" />
-        <origin xyz="0 0 0" />
-	    <xacro:box_inertia_robot m="2" x="0.700" y="0.600" z="0.350"/>
-      </inertial>
-      <visual>
-        <origin xyz="0 0 0" rpy="0 0 0" />
-        <xacro:if value="${hq}">
-          <geometry>
-            <mesh filename="package://rb_theron_description/meshes/bases/mcq_prototype_bottom_cover.dae"/>
-          </geometry>
-        </xacro:if>
-        <xacro:unless value="${hq}">
-          <geometry>
-            <box size="0.700 0.600 0.350"/>
-          </geometry>
-        </xacro:unless>
-        <material name="darkgrey">
-          <color rgba="0.1 0.1 0.1 1"/>
-        </material>
-      </visual>
-      <collision>
-        <origin xyz="0 0 0" rpy="0 0 0 " />
-        <geometry>
-          <mesh filename="package://rb_theron_description/meshes/bases/mcq_prototype_bottom_cover.dae"/>
-        </geometry>
-      </collision>
-    </link> -->
-    <!-- <joint name="${prefix}bottom_cover_joint" type="fixed">
-       <origin rpy="0 0 0" xyz="0 0 0"/>
-       <parent link="${prefix}base_link"/>
-       <child link="${prefix}bottom_cover_link"/>
-    </joint> -->
-    <!-- DOCKING CONTACTS -->
-    <!--joint name="${prefix}base_docking_joint" type="fixed">
-      <origin xyz="0.030 0.000 0.068" rpy="0 0 0 " />
-      <parent link="${prefix}front_cover_link"/>
-      <child link="${prefix}base_docking_contact_link" />
-    </joint-->
-    <!-- DOCKING LINK -->
-    <!--link name="${prefix}base_docking_contact_link" /-->
   </xacro:macro>
 </robot>

File: rb_theron_description/urdf/wheels/castor.urdf.xacro (robot description, xacro)
@@ -33,13 +33,13 @@
         <origin xyz="0 0 0" rpy="0 0 0" />
           <geometry>
-	       <mesh filename="package://rb_theron_description/meshes/wheels/mcq_prototype_base_castor.dae" />
+	       <mesh filename="package://rb_theron_description/meshes/wheels/castor_wheel.stl" />
           </geometry>
       </visual>
-      <collision>
+      <!--collision>
         <origin xyz="0 0 0" rpy="0 0 0" />
           <geometry>
-	       <mesh filename="package://rb_theron_description/meshes/wheels/mcq_prototype_base_castor.dae" />
+	       <mesh filename="package://rb_theron_description/meshes/wheels/castor_wheel.dae" />
           </geometry>
-      </collision>
+      </collision-->
       <inertial>
         <mass value="${caster_support_mass}" />

File: rb_theron_description/urdf/wheels/rubber_wheel.gazebo.xacro (robot description, xacro)
@@ -35,4 +35,8 @@
 			<turnGravityOff>false</turnGravityOff-->
 		</gazebo>
+		<gazebo reference="${prefix}_wheel_tire_link">
+			<material>Gazebo/Gray</material>
+			<turnGravityOff>false</turnGravityOff>
+		</gazebo>
 		<!--gazebo reference="${name}_wheel_link">
 			<kp>500000.0</kp>

File: rb_theron_description/urdf/wheels/rubber_wheel_150.urdf.xacro (robot description, xacro)
@@ -8,5 +8,5 @@
 	<xacro:property name="wheel_radius" value="0.0756" />
 	<xacro:property name="wheel_height" value="0.025" />
-	<xacro:property name="wheel_mass" value="0.25" />
+	<xacro:property name="wheel_mass" value="1" />
 	<!-- in kg-->
 	<xacro:macro name="cylinder_inertia" params="m r h">
@@ -44,4 +44,17 @@
 			</inertial>
 		</link>
+		<joint name="${prefix}_wheel_tire_joint" type="fixed">
+			<parent link="${prefix}_wheel_link"/>
+			<child link="${prefix}_wheel_tire_link"/>
+			<origin xyz="0 0 0" rpy="0 0 0" />
+		</joint>
+		<link name="${prefix}_wheel_tire_link">
+			<visual>
+        <origin xyz="0 0 0" rpy="${M_PI/2} 0 0" />
+				<geometry>
+					<cylinder length="${wheel_height + 0.001}" radius="${wheel_radius * 0.92}" />
+				</geometry>
+			</visual>
+		</link>
 		<xacro:rubber_wheel_transmission prefix="${prefix}" />
 		<xacro:rubber_wheel_gazebo prefix="${prefix}" />

Commit message: description: create an independent base+wheels xacro

File: rb_theron_description/robots/rb_theron.urdf.xacro (robot description, xacro)
@@ -7,11 +7,9 @@
 	<!-- First we import all posible elements defined in the urdf.xacro files. All these elements are defined as macro:xacros -->
 	<!-- Import differential base elements -->
-	<xacro:include filename="$(find rb_theron_description)/urdf/bases/theron_base.urdf.xacro" />
+	<xacro:include filename="$(find rb_theron_description)/robots/rb_theron_base.urdf.xacro" />
 	<!-- Import wheels -->
 	<xacro:include filename="$(find rb_theron_description)/urdf/wheels/rubber_wheel_150.urdf.xacro" />
 	<!-- Import casters -->
 	<xacro:include filename="$(find rb_theron_description)/urdf/wheels/castor.urdf.xacro" />
-	<!-- Import rocker bogie -->
-	<xacro:include filename="$(find rb_theron_description)/urdf/rocker/mcq_prototype_rocker.urdf.xacro" />
 	<!-- Import all available sensors -->
 	<xacro:include filename="$(find robotnik_sensors)/urdf/all_sensors.urdf.xacro" />
@@ -23,7 +21,7 @@
 	<xacro:property name="PI" value="3.1415926535897931"/>
 	<!-- Wheel parameters -->
-	<xacro:property name="wheel_offset_x" value="0" />
+	<!--xacro:property name="wheel_offset_x" value="0" />
 	<xacro:property name="wheel_offset_y" value="0.2516" />
-	<xacro:property name="wheel_offset_z" value="0.0" />
+	<xacro:property name="wheel_offset_z" value="0.0" /-->
 	<!-- Flag to select the high or low quality model -->
 	<xacro:property name="hq" value="true" />
@@ -33,29 +31,10 @@
 	<xacro:arg name="prefix" default="robot_"/>
 	<!-- Here we create the robot elements using the xacro:macros imported at the beggining of this file -->
-	<!-- this property is for the chassis -->
-	<!-- rbogie base -->
-	<xacro:theron_base prefix="$(arg prefix)" publish_bf="true" hq="${hq}" />
+	<!-- base with wheels -->
+	<xacro:rb_theron_base prefix="$(arg prefix)" hq="${hq}" />
 	<!-- Gazebo ros control pluggins -->
 	<xacro:ros_control/>
 	<xacro:gazebo_colors prefix="$(arg prefix)"/>
-	<!-- WHEELS -->
-	<xacro:rubber_wheel prefix="$(arg prefix)right" parent="$(arg prefix)base_link" hq="${hq}">
-		<origin xyz="${wheel_offset_x} ${-wheel_offset_y} ${wheel_offset_z}" rpy="0 0 0"/>
-	</xacro:rubber_wheel>
-	<xacro:rubber_wheel prefix="$(arg prefix)left" parent="$(arg prefix)base_link" hq="${hq}">
-		<origin xyz="${wheel_offset_x} ${wheel_offset_y} ${wheel_offset_z}" rpy="0 0 0"/>
-	</xacro:rubber_wheel>
-	<xacro:caster prefix="$(arg prefix)front_left" parent="$(arg prefix)base_link" hq="${hq}">
-		<origin xyz="0.235 0.1825 0.046" rpy="0 0 0"/>
-	</xacro:caster>
-	<xacro:caster prefix="$(arg prefix)front_right" parent="$(arg prefix)base_link" hq="${hq}">
-		<origin xyz="0.235 -0.1825 0.046" rpy="0 0 0"/>
-	</xacro:caster>
-	<xacro:caster prefix="$(arg prefix)rear_left" parent="$(arg prefix)base_link" hq="${hq}">
-		<origin xyz="-0.235 0.1825 0.046" rpy="0 0 0"/>
-	</xacro:caster>
-	<xacro:caster prefix="$(arg prefix)rear_right" parent="$(arg prefix)base_link" hq="${hq}">
-		<origin xyz="-0.235 -0.1825 0.046" rpy="0 0 0"/>
-	</xacro:caster>
+  <!-- SENSORS -->
   <!-- TODO: Moved 0.01 in x, otherwise the camera is still inside the robot -->
 	<xacro:sensor_orbbec_astra prefix="$(arg prefix)front_rgbd_camera" parent="$(arg prefix)base_link" prefix_topic="front_rgbd_camera">

Commit message: description: update Orbbec camera position

File: rb_theron_description/robots/rb_theron.urdf.xacro (robot description, xacro)
@@ -39,5 +39,5 @@
   <!-- TODO: Moved 0.01 in x, otherwise the camera is still inside the robot -->
 	<xacro:sensor_orbbec_astra prefix="$(arg prefix)front_rgbd_camera" parent="$(arg prefix)base_link" prefix_topic="front_rgbd_camera">
-		<origin xyz="0.3305 0.0 0.1898" rpy="0 0 0"/>
+		<origin xyz="0.3305 0.0 0.1748" rpy="0 0 0"/>
 	</xacro:sensor_orbbec_astra>
 	<xacro:sensor_imu_hector prefix="$(arg prefix)imu" parent="$(arg prefix)base_link">

Commit message: description: add 2x lidar in urdf as default version

File: rb_theron_description/robots/rb_theron.urdf.xacro (robot description, xacro)
@@ -44,6 +44,12 @@
 		<origin xyz="-0.1975 0.0 0.1598" rpy="0 0 0"/>
 	</xacro:sensor_imu_hector>
-	<xacro:sensor_sick_nanoscan3 prefix="$(arg prefix)front_laser" parent="$(arg prefix)base_link" prefix_topic="front_laser" min_angle="-2.0507619" max_angle="2.0507619">
+	<!--xacro:sensor_sick_nanoscan3 prefix="$(arg prefix)front_laser" parent="$(arg prefix)base_link" prefix_topic="front_laser" min_angle="-2.0507619" max_angle="2.0507619">
 		<origin xyz="0.250 0.0 0.1643" rpy="0 3.1416 3.1416"/>
-	</xacro:sensor_sick_nanoscan3>
+	</xacro:sensor_sick_nanoscan3-->
+	<xacro:sensor_sick_tim571 prefix="$(arg prefix)front_laser" parent="$(arg prefix)base_link" prefix_topic="front_laser" min_angle="-2.0507619" max_angle="2.0507619">
+		<origin xyz="0.2675 -0.215 0.1613" rpy="0 -3.1416 2.3562"/>
+	</xacro:sensor_sick_tim571>
+	<xacro:sensor_sick_tim571 prefix="$(arg prefix)rear_laser" parent="$(arg prefix)base_link" prefix_topic="rear_laser" min_angle="-2.0507619" max_angle="2.0507619">
+		<origin xyz="-0.2675 0.215 0.1613" rpy="0 -3.1416 -0.7854"/>
+	</xacro:sensor_sick_tim571>
 </robot>
