Commit message: Added ros2 control and remove prefix
* Now in robot xacro have wheels base and sensor.
* Added ros2 control xacro, for simulation
* Remove package:// in xacro, using find instead
* Remove castor wheel simulation, now are fixed

File: rb_theron_description/robots/rb_theron.urdf.xacro (robot description, xacro)
@@ -4,11 +4,9 @@
   <!-- Imported elements -->
   <!-- ***************** -->
-  <!-- Import differential base elements -->
-  <xacro:include filename="$(find rb_theron_description)/robots/rb_theron_base.urdf.xacro" />
+  <!-- Import RB Theron elements (base + wheels) -->
+  <xacro:include filename="$(find rb_theron_description)/urdf/bases/theron_base.urdf.xacro" />
   <xacro:include filename="$(find rb_theron_description)/urdf/wheels/rubber_wheel_150.urdf.xacro" />
   <xacro:include filename="$(find rb_theron_description)/urdf/wheels/castor.urdf.xacro" />
   <xacro:include filename="$(find robotnik_sensors)/urdf/all_sensors.urdf.xacro" />
-  <!-- Import Gazebo Stuff -->
-  <xacro:include filename="$(find rb_theron_description)/urdf/common.gazebo.xacro" />
   <!-- ***************** -->
   <!-- Global parameters -->
@@ -16,31 +14,52 @@
   <xacro:property name="PI" value="3.1415926535897931"/>
   <!-- Wheel parameters -->
-  <!--xacro:property name="wheel_offset_x" value="0" />
+  <xacro:property name="wheel_offset_x" value="0" />
   <xacro:property name="wheel_offset_y" value="0.2516" />
-  <xacro:property name="wheel_offset_z" value="0.0" /-->
+  <xacro:property name="wheel_offset_z" value="0.0" />
   <!-- Flag to select the high or low quality model -->
   <xacro:property name="hq" value="true" />
-  <xacro:arg name="prefix" default="robot_"/>
-  <xacro:arg name="gpu" default="true"/>
+  <xacro:arg name="robot_id" default="robot"/>
+  <xacro:arg name="robot_id" default="$(arg robot_id)"/>
   <!-- *************** -->
   <!-- Robots Elements -->
   <!-- *************** -->
-  <!-- base with wheels -->
-  <xacro:rb_theron_base prefix="$(arg prefix)" hq="${hq}" />
-  <!-- Gazebo ros control pluggins -->
-  <xacro:ros_control/>
-  <xacro:gazebo_colors prefix="$(arg prefix)"/>
+  <!-- RB Theron -->
+  <xacro:theron_base publish_bf="true" hq="${hq}" />
+  <!-- WHEELS -->
+  <xacro:rubber_wheel prefix="right_" parent="base_link" hq="${hq}">
+    <origin xyz="${wheel_offset_x} ${-wheel_offset_y} ${wheel_offset_z}" rpy="0 0 0"/>
+  </xacro:rubber_wheel>
+  <xacro:rubber_wheel prefix="left_" parent="base_link" hq="${hq}">
+    <origin xyz="${wheel_offset_x} ${wheel_offset_y} ${wheel_offset_z}" rpy="0 0 0"/>
+  </xacro:rubber_wheel>
+  <!-- CASTORS WHEELS -->
+  <xacro:caster prefix="front_left_" parent="base_link" hq="${hq}">
+    <origin xyz="0.235 0.1825 0.046" rpy="0 0 0"/>
+  </xacro:caster>
+  <xacro:caster prefix="front_right_" parent="base_link" hq="${hq}">
+    <origin xyz="0.235 -0.1825 0.046" rpy="0 0 0"/>
+  </xacro:caster>
+  <xacro:caster prefix="rear_left_" parent="base_link" hq="${hq}">
+    <origin xyz="-0.235 0.1825 0.046" rpy="0 0 0"/>
+  </xacro:caster>
+  <xacro:caster prefix="rear_right_" parent="base_link" hq="${hq}">
+    <origin xyz="-0.235 -0.1825 0.046" rpy="0 0 0"/>
+  </xacro:caster>
   <!-- SENSORS -->
-  <xacro:sensor_orbbec_astra prefix="$(arg prefix)front_rgbd_camera" parent="$(arg prefix)base_link" prefix_topic="front_rgbd_camera">
+  <xacro:sensor_orbbec_astra ns="$(arg robot_ns)" prefix="front_rgbd_camera" parent="base_link">
     <origin xyz="0.3305 0.0 0.1748" rpy="0 0 0"/>
   </xacro:sensor_orbbec_astra>
-  <xacro:sensor_imu_hector prefix="$(arg prefix)imu" parent="$(arg prefix)base_link">
+  <xacro:sensor_imu_hector ns="$(arg robot_ns)" prefix="imu" parent="base_link">
     <origin xyz="-0.1975 0.0 0.1598" rpy="0 0 0"/>
   </xacro:sensor_imu_hector>
-  <xacro:sensor_sick_tim571 prefix="$(arg prefix)front_laser" parent="$(arg prefix)base_link" prefix_topic="front_laser" min_angle="-2.0507619" max_angle="2.0507619" gpu="$(arg gpu)">
+  <xacro:sensor_sick_tim571 ns="$(arg robot_ns)" prefix="front_laser" parent="base_link">
     <origin xyz="0.2675 -0.215 0.1613" rpy="0 -3.1416 2.3562"/>
   </xacro:sensor_sick_tim571>
-  <xacro:sensor_sick_tim571 prefix="$(arg prefix)rear_laser" parent="$(arg prefix)base_link" prefix_topic="rear_laser" min_angle="-2.0507619" max_angle="2.0507619" gpu="$(arg gpu)">
+  <xacro:sensor_sick_tim571 ns="$(arg robot_ns)" prefix="rear_laser" parent="base_link">
     <origin xyz="-0.2675 0.215 0.1613" rpy="0 -3.1416 -0.7854"/>
   </xacro:sensor_sick_tim571>
+  <!-- Gazebo ros control plugins -->
+  <xacro:arg name="config_controllers" default=""/>
+  <xacro:include filename="$(find rb_theron_description)/urdf/ros2_control.urdf.xacro"/>
+  <xacro:ros2_control/>
 </robot>

File: rb_theron_description/urdf/bases/theron_base.urdf.xacro (robot description, xacro)
@@ -1,18 +1,18 @@
 <?xml version="1.0"?>
 <robot name="theron_base" xmlns:xacro="http://www.ros.org/wiki/xacro">
-  <xacro:macro name="theron_base" params="prefix publish_bf hq">
+  <xacro:macro name="theron_base" params="publish_bf hq">
     <xacro:property name="PI" value="3.1415926535897931"/>
     <!-- xacro:property name="wheel_width" value="0.150" / -->
     <!-- BASE FOOTPRINT -->
     <xacro:if value="${publish_bf}">
-      <link name="${prefix}base_footprint" />
-      <joint name="${prefix}base_footprint_joint" type="fixed">
-        <origin xyz="0 0 ${wheel_radius - wheel_offset_z}" rpy="0 0 0" />
-        <parent link="${prefix}base_footprint"/>
-        <child link="${prefix}base_link" />
+      <link name="base_footprint"/>
+      <joint name="base_footprint_joint" type="fixed">
+        <origin xyz="0 0 ${wheel_radius - wheel_offset_z}" rpy="0 0 0"/>
+        <parent link="base_footprint"/>
+        <child link="base_link" />
       </joint>
     </xacro:if>
     <!-- BASE_LINK -->
-    <link name="${prefix}base_link">
+    <link name="base_link">
       <inertial>
         <mass value="45" />
@@ -24,5 +24,5 @@
         <xacro:if value="${hq}">
           <geometry>
-            <mesh filename="package://rb_theron_description/meshes/bases/theron_base.stl"/>
+            <mesh filename="file://$(find rb_theron_description)/meshes/bases/theron_base.stl"/>
           </geometry>
         </xacro:if>
@@ -39,5 +39,5 @@
         <origin xyz="0 0 0.005" rpy="0 0 0 " />
         <geometry>
-          <mesh filename="package://rb_theron_description/meshes/bases/theron_base.dae"/>
+          <mesh filename="file://$(find rb_theron_description)/meshes/bases/theron_base.dae"/>
         </geometry>
       </collision>

File: rb_theron_description/urdf/pole/mcq_pole.urdf.xacro (robot description, xacro)
@@ -23,5 +23,5 @@
         <origin xyz="0 0 0" rpy="0 0 0" />
           <geometry>
-            <mesh filename="package://rb_theron_description/meshes/pole/mcq_pole.stl"/>
+            <mesh filename="file://$(find rb_theron_description)/meshes/pole/mcq_pole.stl"/>
           </geometry>
         <material name="darkgrey">
@@ -32,5 +32,5 @@
         <origin xyz="0 0 0" rpy="0 0 0 " />
         <geometry>
-          <mesh filename="package://rb_theron_description/meshes/pole/mcq_pole.stl"/>
+          <mesh filename="file://$(find rb_theron_description)/meshes/pole/mcq_pole.stl"/>
         </geometry>
       </collision>

File: rb_theron_description/urdf/pole/simple_pole.urdf.xacro (robot description, xacro)
@@ -23,5 +23,5 @@
         <origin xyz="0 0 0" rpy="0 0 0" />
           <geometry>
-            <mesh filename="package://rb_theron_description/meshes/pole/simple_pole.dae"/>
+            <mesh filename="file://$(find rb_theron_description)/meshes/pole/simple_pole.dae"/>
           </geometry>
         <material name="darkgrey">
@@ -32,5 +32,5 @@
         <origin xyz="0 0 0" rpy="0 0 0 " />
         <geometry>
-          <mesh filename="package://rb_theron_description/meshes/pole/simple_pole.dae"/>
+          <mesh filename="file://$(find rb_theron_description)/meshes/pole/simple_pole.dae"/>
         </geometry>
       </collision>

File: rb_theron_description/urdf/rocker/mcq_prototype_rocker.urdf.xacro (robot description, xacro)
@@ -36,10 +36,10 @@
           <xacro:if value="${reflect}">
             <geometry>
-            <mesh filename="package://rb_theron_description/meshes/rocker/mcq_prototype_rocker_r.dae" />
+            <mesh filename="file://$(find rb_theron_description)/meshes/rocker/mcq_prototype_rocker_r.dae" />
             </geometry>
           </xacro:if>
           <xacro:unless value="${reflect}">
             <geometry>
-              <mesh filename="package://rb_theron_description/meshes/rocker/mcq_prototype_rocker_l.dae" />
+              <mesh filename="file://$(find rb_theron_description)/meshes/rocker/mcq_prototype_rocker_l.dae" />
             </geometry>
       </xacro:unless>
@@ -49,10 +49,10 @@
           <xacro:if value="${reflect}">
             <geometry>
-            <mesh filename="package://rb_theron_description/meshes/rocker/mcq_prototype_rocker_r.dae" />
+            <mesh filename="file://$(find rb_theron_description)/meshes/rocker/mcq_prototype_rocker_r.dae" />
             </geometry>
           </xacro:if>
           <xacro:unless value="${reflect}">
             <geometry>
-              <mesh filename="package://rb_theron_description/meshes/rocker/mcq_prototype_rocker_l.dae" />
+              <mesh filename="file://$(find rb_theron_description)/meshes/rocker/mcq_prototype_rocker_l.dae" />
             </geometry>
       </xacro:unless>

File: rb_theron_description/urdf/wheels/castor.urdf.xacro (robot description, xacro)
@@ -19,13 +19,9 @@
   </xacro:macro>
   <xacro:macro name="caster" params="prefix parent *origin hq">
-  <!--CASTER SUPPORT -->
-  <joint name="${prefix}joint_support" type="continuous">
+    <!--CASTER SUPPORT -->
+    <joint name="${prefix}joint_support" type="fixed">
+      <xacro:insert_block name="origin" />
       <parent link="${parent}"/>
       <child link="${prefix}support"/>
-      <xacro:insert_block name="origin" />
-      <axis xyz="0 0 1" rpy="0 ${M_PI} 0" />
-      <limit effort="100" velocity="100"/>
-      <!-- joint_properties damping="1.5" friction="1.5"/ -->
-      <dynamics damping="0" friction="0.01"/>
     </joint>
     <link name="${prefix}support">
@@ -33,13 +29,13 @@
         <origin xyz="0 0 0" rpy="0 0 0" />
           <geometry>
-         <mesh filename="package://rb_theron_description/meshes/wheels/castor_wheel.stl" />
+         <mesh filename="file://$(find rb_theron_description)/meshes/wheels/castor_wheel.stl" />
           </geometry>
       </visual>
-      <!--collision>
-        <origin xyz="0 0 0" rpy="0 0 0" />
-          <geometry>
-         <mesh filename="package://rb_theron_description/meshes/wheels/castor_wheel.dae" />
-          </geometry>
-      </collision-->
+      <collision>
+        <origin xyz="0 0 ${caster_wheel_offset_z}" rpy="0 0 0" />
+        <geometry>
+          <sphere radius="${caster_radius}"/>
+        </geometry>
+      </collision>
       <inertial>
         <mass value="${caster_support_mass}" />
@@ -48,93 +44,11 @@
       </inertial>
     </link>
-  <!--CASTER WHEEL -->
-  <!-- xacro:caster_wheel prefix="${prefix}" parent="${prefix}support" hq="${hq}" -->
-  <xacro:caster_wheel prefix="${prefix}" parent="${prefix}support" hq="${hq}">
-    <origin xyz="${caster_wheel_offset_x} ${caster_wheel_offset_y} ${caster_wheel_offset_z}" rpy="0 0 0"/>
-   </xacro:caster_wheel>
- </xacro:macro>
- <xacro:macro name="caster_wheel" params="prefix parent *origin hq">
-     <joint name="${prefix}joint_wheel" type="continuous">
-       <parent link="${parent}"/>
-       <child link="${prefix}wheel"/>
-       <xacro:insert_block name="origin" />
-       <axis xyz="0 1 0" rpy="0 0 0" />
-       <limit effort="100" velocity="100"/>
-       <joint_properties damping="0.1" friction="0.1"/>
-    </joint>
-    <link name="${prefix}wheel">
-      <visual>
-        <!-- HIGH RESOLUTION WHEELS -->
-     <!-- xacro:if value="${hq}">
-          <origin xyz="0 0 0" rpy="0 0 0" />
-          <geometry>
-    <mesh filename="package://rb_theron_description/meshes/wheels/mcq_prototype_castor_wheel.dae" />
-          </geometry>
-        </xacro:if -->
-       <!-- LOW RESOLUTION WHEELS -->
-       <!-- xacro:unless value="${hq}" -->
-          <origin xyz="0 0 0" rpy="${M_PI/2} 0 0" />
-          <geometry>
-            <cylinder length="${caster_height}" radius="${caster_radius}" />
-            <!-- sphere radius="${caster_radius}"/ -->
-          </geometry>
-        <!-- /xacro:unless -->
-      </visual>
-     <collision>
-    <origin xyz="0 0 0" rpy="${M_PI/2} 0 0" />
-    <!-- origin xyz="0 0 0" rpy="0 0 0" / -->
-        <geometry>
-      <!-- mesh filename="package://rb_theron_description/meshes/wheels/mcq_prototype_castor_wheel.dae" / -->
-          <cylinder length="${caster_height}" radius="${caster_radius}" />
-          <!-- sphere radius="${caster_radius}"/ -->
-        </geometry>
-    <surface>
-          <bounce restitution_coefficient = "1"/>
-    </surface>
-      </collision>
-      <inertial>
-        <mass value="${caster_mass}" />
-        <origin xyz="0 0 0" />
-        <xacro:cylinder_inertia  m="${caster_mass}" r="${caster_radius}" h="${caster_height}" />
-      </inertial>
-    </link>
-  <!-- Transmission is important to link the joints and the controller -->
-    <transmission name="${prefix}support_joint_trans">
-      <type>transmission_interface/SimpleTransmission</type>
-      <joint name="${prefix}joint_support">
-          <hardwareInterface>hardware_interface/EffortJointInterface</hardwareInterface>
-      </joint>
-      <actuator name="${prefix}support_joint_motor">
-        <mechanicalReduction>1</mechanicalReduction>
-        <motorTorqueConstant>1</motorTorqueConstant>
-      </actuator>
-    </transmission>
-    <transmission name="${prefix}wheel_joint_trans">
-      <type>transmission_interface/SimpleTransmission</type>
-      <joint name="${prefix}joint_wheel">
-          <hardwareInterface>hardware_interface/EffortJointInterface</hardwareInterface>
-      </joint>
-      <actuator name="${prefix}wheel_joint_motor">
-        <mechanicalReduction>1</mechanicalReduction>
-    <motorTorqueConstant>1</motorTorqueConstant>
-      </actuator>
-    </transmission>
-    <!-- gazebo reference="${prefix}support">
-      <mu1 value="5.0"/>
-      <mu2 value="0.5"/>
-      <kp value="10000000.0" />
-      <kd value="1.0" />
-      <fdir1 value="1 0 0"/>
-      <turnGravityOff>false</turnGravityOff>
-    </gazebo -->
-     <gazebo reference="${prefix}_wheel">
-      <mu1 value="100.0"/>
-      <mu2 value="100.0"/>
-      <!-- kp value="10000000.0" / -->
-      <kp value="100000.0" />
-      <kd value="100.0" />
-      <!-- fdir1 value="1 0 0"/ -->
-      <material>Gazebo/Black</material>
-      <turnGravityOff>false</turnGravityOff>
+    <gazebo reference="${prefix}support">
+      <mu1>0.001</mu1>
+      <mu2>0.001</mu2>
+      <kp>2.75e7</kp>
+      <kd>8.25e1</kd>
+      <fdir1>0 0 0</fdir1>
+      <maxContacts>4</maxContacts>
     </gazebo>
  </xacro:macro>

File: rb_theron_description/urdf/wheels/rubber_wheel_150.urdf.xacro (robot description, xacro)
@@ -15,7 +15,7 @@
     <xacro:macro name="rubber_wheel" params="prefix parent *origin hq">
         <!--WHEEL TIRE -->
-        <joint name="${prefix}_wheel_joint" type="continuous">
+        <joint name="${prefix}wheel_joint" type="continuous">
             <parent link="${parent}"/>
-            <child link="${prefix}_wheel_link"/>
+            <child link="${prefix}wheel_link"/>
             <xacro:insert_block name="origin" />
             <axis xyz="0 1 0" rpy="0 0 0" />
@@ -23,5 +23,5 @@
             <joint_properties damping="0.0" friction="0.0"/>
         </joint>
-        <link name="${prefix}_wheel_link">
+        <link name="${prefix}wheel_link">
             <visual>
                 <!-- HIGH RESOLUTION WHEELS -->
@@ -44,10 +44,10 @@
             </inertial>
         </link>
-        <joint name="${prefix}_wheel_tire_joint" type="fixed">
-            <parent link="${prefix}_wheel_link"/>
-            <child link="${prefix}_wheel_tire_link"/>
+        <joint name="${prefix}wheel_tire_joint" type="fixed">
+            <parent link="${prefix}wheel_link"/>
+            <child link="${prefix}wheel_tire_link"/>
             <origin xyz="0 0 0" rpy="0 0 0" />
         </joint>
-        <link name="${prefix}_wheel_tire_link">
+        <link name="${prefix}wheel_tire_link">
             <visual>
         <origin xyz="0 0 0" rpy="${M_PI/2} 0 0" />

Commit message: Added 3d lidar and gpu option

File: rb_theron_description/robots/rb_theron.urdf.xacro (robot description, xacro)
@@ -20,5 +20,5 @@
   <xacro:property name="hq" value="true" />
   <xacro:arg name="robot_id" default="robot"/>
-  <xacro:arg name="robot_id" default="$(arg robot_id)"/>
+	<xacro:arg name="gpu" default="true"/>
   <!-- *************** -->
   <!-- Robots Elements -->
@@ -53,10 +53,13 @@
     <origin xyz="-0.1975 0.0 0.1598" rpy="0 0 0"/>
   </xacro:sensor_imu_hector>
-  <xacro:sensor_sick_tim571 ns="$(arg robot_ns)" prefix="front_laser" parent="base_link">
+  <xacro:sensor_sick_tim571 ns="$(arg robot_ns)" prefix="front_laser" parent="base_link" gpu="$(arg gpu)">
     <origin xyz="0.2675 -0.215 0.1613" rpy="0 -3.1416 2.3562"/>
   </xacro:sensor_sick_tim571>
-  <xacro:sensor_sick_tim571 ns="$(arg robot_ns)" prefix="rear_laser" parent="base_link">
+  <xacro:sensor_sick_tim571 ns="$(arg robot_ns)" prefix="rear_laser" parent="base_link" gpu="$(arg gpu)">
     <origin xyz="-0.2675 0.215 0.1613" rpy="0 -3.1416 -0.7854"/>
   </xacro:sensor_sick_tim571>
+  <xacro:sensor_velodyne_vlp16 ns="$(arg robot_ns)" prefix="top_laser_" parent="base_link" gpu="$(arg gpu)">
+    <origin xyz="0 0 0.3" rpy="0 0 0"/>
+  </xacro:sensor_velodyne_vlp16>
   <!-- Gazebo ros control plugins -->
   <xacro:arg name="config_controllers" default=""/>
