Commit message: Add use_sim variable for castor wheel simulation

File: rb_theron_description/robots/rb_theron.urdf.xacro (robot description, xacro)
@@ -10,6 +10,4 @@
 	<!-- Import wheels -->
 	<xacro:include filename="$(find rb_theron_description)/urdf/wheels/rubber_wheel_150.urdf.xacro" />
-	<!-- Import casters -->
-	<xacro:include filename="$(find rb_theron_description)/urdf/wheels/castor.urdf.xacro" />
 	<!-- Import all available sensors -->
 	<xacro:include filename="$(find robotnik_sensors)/urdf/all_sensors.urdf.xacro" />
@@ -31,7 +29,8 @@
 	<xacro:arg name="prefix" default="robot_"/>
 	<xacro:arg name="gpu" default="true"/>
+	<xacro:arg name="use_sim" default="false"/>
 	<!-- Here we create the robot elements using the xacro:macros imported at the beggining of this file -->
 	<!-- base with wheels -->
-	<xacro:rb_theron_base prefix="$(arg prefix)" hq="${hq}" />
+	<xacro:rb_theron_base prefix="$(arg prefix)" hq="${hq}" use_sim="$(arg use_sim)"/>
 	<!-- Gazebo ros control pluggins -->
 	<xacro:ros_control/>

File: rb_theron_description/robots/rb_theron_base.urdf.xacro (robot description, xacro)
@@ -25,5 +25,5 @@
 	<!-- Robots Elements -->
 	<!-- *************** -->
-  <xacro:macro name="rb_theron_base" params="prefix hq">
+  <xacro:macro name="rb_theron_base" params="prefix hq use_sim">
     <!-- rbogie base -->
   	<xacro:theron_base prefix="${prefix}" publish_bf="true" hq="${hq}" />
@@ -37,16 +37,16 @@
   	</xacro:rubber_wheel>
 <!-- Castor wheels-->
-  	<xacro:caster prefix="${prefix}front_left" parent="${prefix}base_link" hq="${hq}">
-  		<origin xyz="0.235 0.1825 0.0448" rpy="0 0 0"/>
-  	</xacro:caster>
-  	<xacro:caster prefix="${prefix}front_right" parent="${prefix}base_link" hq="${hq}">
-  		<origin xyz="0.235 -0.1825 0.0448" rpy="0 0 0"/>
-  	</xacro:caster>
-  	<xacro:caster prefix="${prefix}rear_left" parent="${prefix}base_link" hq="${hq}">
-  		<origin xyz="-0.235 0.1825 0.0448" rpy="0 0 0"/>
-  	</xacro:caster>
-  	<xacro:caster prefix="${prefix}rear_right" parent="${prefix}base_link" hq="${hq}">
-  		<origin xyz="-0.235 -0.1825 0.0448" rpy="0 0 0"/>
-  	</xacro:caster>
+	<xacro:caster prefix="${prefix}front_left" parent="${prefix}base_link" hq="${hq}" use_sim="$(arg use_sim)">
+		<origin xyz="0.235 0.1825 0.0448" rpy="0 0 0"/>
+	</xacro:caster>
+	<xacro:caster prefix="${prefix}front_right" parent="${prefix}base_link" hq="${hq}" use_sim="$(arg use_sim)">
+		<origin xyz="0.235 -0.1825 0.0448" rpy="0 0 0"/>
+	</xacro:caster>
+	<xacro:caster prefix="${prefix}rear_left" parent="${prefix}base_link" hq="${hq}" use_sim="$(arg use_sim)">
+		<origin xyz="-0.235 0.1825 0.0448" rpy="0 0 0"/>
+	</xacro:caster>
+	<xacro:caster prefix="${prefix}rear_right" parent="${prefix}base_link" hq="${hq}" use_sim="$(arg use_sim)">
+		<origin xyz="-0.235 -0.1825 0.0448" rpy="0 0 0"/>
+	</xacro:caster>
   </xacro:macro>
 </robot>

File: rb_theron_description/robots/rb_theron_elevator.urdf.xacro (robot description, xacro)
@@ -10,6 +10,4 @@
 	<!-- Import wheels -->
 	<xacro:include filename="$(find rb_theron_description)/urdf/wheels/rubber_wheel_150.urdf.xacro" />
-	<!-- Import casters -->
-	<xacro:include filename="$(find rb_theron_description)/urdf/wheels/castor.urdf.xacro" />
 	<!-- Import all available sensors -->
 	<xacro:include filename="$(find robotnik_sensors)/urdf/all_sensors.urdf.xacro" />
@@ -37,4 +35,5 @@
 	<xacro:arg name="ros_planar_move_plugin" default="false"/>
 	<xacro:arg name="gpu" default="false"/>
+	<xacro:arg name="use_sim" default="false"/>
 	<!-- *************** -->
 	<!-- Robots Elements -->
@@ -43,5 +42,5 @@
 	<!-- Here we create the robot elements using the xacro:macros imported at the beggining of this file -->
 	<!-- base with wheels -->
-	<xacro:rb_theron_base prefix="$(arg prefix)" hq="${hq}" />
+	<xacro:rb_theron_base prefix="$(arg prefix)" hq="${hq}" use_sim="$(arg use_sim)"/>
 	<!-- Gazebo ros control pluggins -->
 	<xacro:ros_control/>

File: rb_theron_description/urdf/wheels/castor.urdf.xacro (robot description, xacro)
@@ -18,15 +18,28 @@
               izz="${m*r*r/2}" />
   </xacro:macro>
-  <xacro:macro name="caster" params="prefix parent *origin hq">
+  <xacro:macro name="caster" params="prefix parent *origin hq use_sim">
   <!--CASTER SUPPORT -->
-  <joint name="${prefix}joint_support" type="fixed">
+  <xacro:if value="${use_sim}">
+    <joint name="${prefix}joint_support" type="continuous">
       <parent link="${parent}"/>
       <child link="${prefix}_support"/>
       <xacro:insert_block name="origin" />
       <axis xyz="0 0 1" rpy="0 ${M_PI} 0" />
-      <!-- <limit effort="100" velocity="100"/> -->
+      <limit effort="100" velocity="100"/>
       <!-- joint_properties damping="1.5" friction="1.5"/ -->
       <dynamics damping="0" friction="0.01"/>
     </joint>
+  </xacro:if>
+  <xacro:unless value="${use_sim}">
+    <joint name="${prefix}joint_support" type="fixed">
+        <parent link="${parent}"/>
+        <child link="${prefix}_support"/>
+        <xacro:insert_block name="origin" />
+        <axis xyz="0 0 1" rpy="0 ${M_PI} 0" />
+        <!-- <limit effort="100" velocity="100"/> -->
+        <!-- joint_properties damping="1.5" friction="1.5"/ -->
+        <dynamics damping="0" friction="0.01"/>
+      </joint>
+  </xacro:unless>
     <link name="${prefix}_support">
       <visual>
@@ -50,9 +63,20 @@
   <!--CASTER WHEEL -->
   <!-- xacro:caster_wheel prefix="${prefix}" parent="${prefix}_support" hq="${hq}" -->
-  <xacro:caster_wheel prefix="${prefix}" parent="${prefix}_support" hq="${hq}">
+  <xacro:caster_wheel prefix="${prefix}" parent="${prefix}_support" hq="${hq}" use_sim="$(arg use_sim)">
 		<origin xyz="${caster_wheel_offset_x} ${caster_wheel_offset_y} ${caster_wheel_offset_z}" rpy="0 0 0"/>
    </xacro:caster_wheel>
  </xacro:macro>
- <xacro:macro name="caster_wheel" params="prefix parent *origin hq">
+ <xacro:macro name="caster_wheel" params="prefix parent *origin hq use_sim">
+  <xacro:if value="${use_sim}">
+    <joint name="${prefix}joint_wheel" type="continuous">
+      <parent link="${parent}"/>
+      <child link="${prefix}_wheel"/>
+      <insert_block name="origin" />
+      <axis xyz="0 1 0" rpy="0 0 0" />
+      <limit effort="100" velocity="100"/>
+      <joint_properties damping="0.1" friction="0.1"/>
+   </joint>
+  </xacro:if>
+  <xacro:unless value="${use_sim}">
      <joint name="${prefix}joint_wheel" type="fixed">
        <parent link="${parent}"/>
@@ -63,4 +87,5 @@
        <joint_properties damping="0.1" friction="0.1"/>
     </joint>
+  </xacro:unless>
     <link name="${prefix}_wheel">
       <visual>
@@ -99,5 +124,6 @@
       </inertial>
     </link>
-  <!-- Transmission is important to link the joints and the controller
+  <!-- Transmission is important to link the joints and the controller-->
+  <xacro:if value="${use_sim}">
     <transmission name="${prefix}_support_joint_trans">
       <type>transmission_interface/SimpleTransmission</type>
@@ -120,5 +146,5 @@
       </actuator>
     </transmission>
-  -->
+  </xacro:if>
     <gazebo reference="${prefix}_support">
 			<mu1 value="5.0"/>

Commit message: Corrected harcoded ros_control robot description
- fixes #8

File: rb_theron_description/robots/rb_theron.urdf.xacro (robot description, xacro)
@@ -34,5 +34,5 @@
 	<xacro:rb_theron_base prefix="$(arg prefix)" hq="${hq}" use_sim="$(arg use_sim)"/>
 	<!-- Gazebo ros control pluggins -->
-	<xacro:ros_control/>
+	<xacro:ros_control namespace="$(arg namespace)"/>
 	<xacro:gazebo_colors prefix="$(arg prefix)"/>
   <!-- SENSORS -->

File: rb_theron_description/urdf/common.gazebo.xacro (robot description, xacro)
@@ -2,9 +2,9 @@
 <robot xmlns:xacro="http://www.ros.org/wiki/xacro">
 	<!-- ROS CONTROL GAZEBO PLUGIN -->
-	<xacro:macro name="ros_control">
+	<xacro:macro name="ros_control" params="namespace:=robot">
 		<gazebo>
 			<plugin name="ros_control" filename="libgazebo_ros_control.so">
 				<!--robotNamespace>/robot</robotNamespace-->
-				<robotParam>robot/robot_description</robotParam>
+				<robotParam>${namespace}/robot_description</robotParam>
 				<controlPeriod>0.001</controlPeriod>
 				<robotSimType>gazebo_ros_control/DefaultRobotHWSim</robotSimType>

Commit message: Update default rb_theron base

File: rb_theron_description/robots/rb_theron.urdf.xacro (robot description, xacro)
@@ -45,20 +45,32 @@
   	</xacro:if>
 	<xacro:gazebo_colors prefix="$(arg prefix)"/>
-  <!-- SENSORS -->
+<!-- SENSORS -->
   <!-- TODO: Moved 0.01 in x, otherwise the camera is still inside the robot -->
-	<xacro:sensor_orbbec_astra prefix="$(arg prefix)front_rgbd_camera" parent="$(arg prefix)base_link" prefix_topic="front_rgbd_camera">
+	<!--xacro:sensor_orbbec_astra prefix="$(arg prefix)front_rgbd_camera" parent="$(arg prefix)base_link" prefix_topic="front_rgbd_camera">
 		<origin xyz="0.3305 0.0 0.1748" rpy="0 0 0"/>
-	</xacro:sensor_orbbec_astra>
+	</xacro:sensor_orbbec_astra-->
+	<xacro:sensor_intel_d435 prefix="$(arg prefix)front_rgbd_camera" parent="$(arg prefix)base_link" prefix_topic="front_rgbd_camera">
+		<origin xyz="0.3045 0.0 0.1898" rpy="0 0 0"/>
+	</xacro:sensor_intel_d435>
+	<xacro:sensor_intel_d435 prefix="$(arg prefix)rear_rgbd_camera" parent="$(arg prefix)base_link" prefix_topic="rear_rgbd_camera">
+		<origin xyz="-0.3045 0.0 0.1158" rpy="0 0 3.1416"/>
+	</xacro:sensor_intel_d435>
 	<xacro:sensor_imu_hector prefix="$(arg prefix)imu" parent="$(arg prefix)base_link">
 		<origin xyz="-0.1975 0.0 0.1598" rpy="0 0 0"/>
 	</xacro:sensor_imu_hector>
+	<xacro:sensor_hokuyo_ust20lx prefix="$(arg prefix)front_laser" parent="$(arg prefix)base_link" prefix_topic="front_laser" min_angle="-2.0507619" max_angle="2.0507619">
+		<origin xyz="0.2675 -0.215 0.1613" rpy="0 -3.1416 2.3562"/>
+	</xacro:sensor_hokuyo_ust20lx>
+	<xacro:sensor_hokuyo_ust20lx prefix="$(arg prefix)rear_laser" parent="$(arg prefix)base_link" prefix_topic="rear_laser" min_angle="-2.0507619" max_angle="2.0507619">
+		<origin xyz="-0.2675 0.215 0.1613" rpy="0 -3.1416 -0.7854"/>
+	</xacro:sensor_hokuyo_ust20lx>
 	<!--xacro:sensor_sick_nanoscan3 prefix="$(arg prefix)front_laser" parent="$(arg prefix)base_link" prefix_topic="front_laser" min_angle="-2.0507619" max_angle="2.0507619">
 		<origin xyz="0.250 0.0 0.1643" rpy="0 3.1416 3.1416"/>
 	</xacro:sensor_sick_nanoscan3-->
-	<xacro:sensor_sick_tim571 prefix="$(arg prefix)front_laser" parent="$(arg prefix)base_link" prefix_topic="front_laser" min_angle="-2.0507619" max_angle="2.0507619" gpu="$(arg gpu)">
+	<!--xacro:sensor_sick_tim571 prefix="$(arg prefix)front_laser" parent="$(arg prefix)base_link" prefix_topic="front_laser" min_angle="-2.0507619" max_angle="2.0507619">
 		<origin xyz="0.2675 -0.215 0.1613" rpy="0 -3.1416 2.3562"/>
-	</xacro:sensor_sick_tim571>
-	<xacro:sensor_sick_tim571 prefix="$(arg prefix)rear_laser" parent="$(arg prefix)base_link" prefix_topic="rear_laser" min_angle="-2.0507619" max_angle="2.0507619" gpu="$(arg gpu)">
+	</xacro:sensor_sick_tim571-->
+	<!--xacro:sensor_sick_tim571 prefix="$(arg prefix)rear_laser" parent="$(arg prefix)base_link" prefix_topic="rear_laser" min_angle="-2.0507619" max_angle="2.0507619">
 		<origin xyz="-0.2675 0.215 0.1613" rpy="0 -3.1416 -0.7854"/>
-	</xacro:sensor_sick_tim571>
+	</xacro:sensor_sick_tim571-->
 </robot>

Commit message: Update default rb_theron base

File: rb_theron_description/robots/rb_theron.urdf.xacro (robot description, xacro)
@@ -36,20 +36,32 @@
 	<xacro:ros_control namespace="$(arg namespace)"/>
 	<xacro:gazebo_colors prefix="$(arg prefix)"/>
-  <!-- SENSORS -->
+<!-- SENSORS -->
   <!-- TODO: Moved 0.01 in x, otherwise the camera is still inside the robot -->
-	<xacro:sensor_orbbec_astra prefix="$(arg prefix)front_rgbd_camera" parent="$(arg prefix)base_link" prefix_topic="front_rgbd_camera">
+	<!--xacro:sensor_orbbec_astra prefix="$(arg prefix)front_rgbd_camera" parent="$(arg prefix)base_link" prefix_topic="front_rgbd_camera">
 		<origin xyz="0.3305 0.0 0.1748" rpy="0 0 0"/>
-	</xacro:sensor_orbbec_astra>
+	</xacro:sensor_orbbec_astra-->
+	<xacro:sensor_intel_d435 prefix="$(arg prefix)front_rgbd_camera" parent="$(arg prefix)base_link" prefix_topic="front_rgbd_camera">
+		<origin xyz="0.3045 0.0 0.1898" rpy="0 0 0"/>
+	</xacro:sensor_intel_d435>
+	<xacro:sensor_intel_d435 prefix="$(arg prefix)rear_rgbd_camera" parent="$(arg prefix)base_link" prefix_topic="rear_rgbd_camera">
+		<origin xyz="-0.3045 0.0 0.1158" rpy="0 0 3.1416"/>
+	</xacro:sensor_intel_d435>
 	<xacro:sensor_imu_hector prefix="$(arg prefix)imu" parent="$(arg prefix)base_link">
 		<origin xyz="-0.1975 0.0 0.1598" rpy="0 0 0"/>
 	</xacro:sensor_imu_hector>
+	<xacro:sensor_hokuyo_ust20lx prefix="$(arg prefix)front_laser" parent="$(arg prefix)base_link" prefix_topic="front_laser" min_angle="-2.0507619" max_angle="2.0507619">
+		<origin xyz="0.2675 -0.215 0.1613" rpy="0 -3.1416 2.3562"/>
+	</xacro:sensor_hokuyo_ust20lx>
+	<xacro:sensor_hokuyo_ust20lx prefix="$(arg prefix)rear_laser" parent="$(arg prefix)base_link" prefix_topic="rear_laser" min_angle="-2.0507619" max_angle="2.0507619">
+		<origin xyz="-0.2675 0.215 0.1613" rpy="0 -3.1416 -0.7854"/>
+	</xacro:sensor_hokuyo_ust20lx>
 	<!--xacro:sensor_sick_nanoscan3 prefix="$(arg prefix)front_laser" parent="$(arg prefix)base_link" prefix_topic="front_laser" min_angle="-2.0507619" max_angle="2.0507619">
 		<origin xyz="0.250 0.0 0.1643" rpy="0 3.1416 3.1416"/>
 	</xacro:sensor_sick_nanoscan3-->
-	<xacro:sensor_sick_tim571 prefix="$(arg prefix)front_laser" parent="$(arg prefix)base_link" prefix_topic="front_laser" min_angle="-2.0507619" max_angle="2.0507619" gpu="$(arg gpu)">
+	<!--xacro:sensor_sick_tim571 prefix="$(arg prefix)front_laser" parent="$(arg prefix)base_link" prefix_topic="front_laser" min_angle="-2.0507619" max_angle="2.0507619">
 		<origin xyz="0.2675 -0.215 0.1613" rpy="0 -3.1416 2.3562"/>
-	</xacro:sensor_sick_tim571>
-	<xacro:sensor_sick_tim571 prefix="$(arg prefix)rear_laser" parent="$(arg prefix)base_link" prefix_topic="rear_laser" min_angle="-2.0507619" max_angle="2.0507619" gpu="$(arg gpu)">
+	</xacro:sensor_sick_tim571-->
+	<!--xacro:sensor_sick_tim571 prefix="$(arg prefix)rear_laser" parent="$(arg prefix)base_link" prefix_topic="rear_laser" min_angle="-2.0507619" max_angle="2.0507619">
 		<origin xyz="-0.2675 0.215 0.1613" rpy="0 -3.1416 -0.7854"/>
-	</xacro:sensor_sick_tim571>
+	</xacro:sensor_sick_tim571-->
 </robot>
