Commit message: Changed tabs to spaces and removed spaces

File: rb_theron_description/urdf/bases/theron_base.urdf.xacro (robot description, xacro)
@@ -1,24 +1,10 @@
 <?xml version="1.0"?>
-<robot name="rbogie_base"
-  xmlns:xacro="http://www.ros.org/wiki/xacro">
-<!--macro name="box_inertia_robot" params="m x y z">
-        <inertia  ixx="${m*(y*y+z*z)/12}" ixy = "0" ixz = "0"
-                  iyy="${m*(x*x+z*z)/12}" iyz = "0"
-                  izz="${m*(x*x+z*z)/12}" />
-</macro-->
+<robot name="theron_base" xmlns:xacro="http://www.ros.org/wiki/xacro">
   <xacro:macro name="theron_base" params="prefix publish_bf hq">
-    <!-- Robot mechanical and motor parameters -->
     <xacro:property name="PI" value="3.1415926535897931"/>
     <!-- xacro:property name="wheel_width" value="0.150" / -->
     <!-- BASE FOOTPRINT -->
     <xacro:if value="${publish_bf}">
-      <link name="${prefix}base_footprint">
-        <visual>
-          <origin xyz="0 0 0" rpy="0 0 0" />
-          <geometry>
-            <box size="0.001 0.001 0.001" />
-          </geometry>
-        </visual>
-      </link>
+      <link name="${prefix}base_footprint" />
       <joint name="${prefix}base_footprint_joint" type="fixed">
         <origin xyz="0 0 ${wheel_radius - wheel_offset_z}" rpy="0 0 0" />
@@ -30,8 +16,8 @@
     <link name="${prefix}base_link">
       <inertial>
-      <mass value="45" />
-      <origin xyz="0.0 0.0 0.0" />
-      <xacro:solid_cuboid_inertia m="45" w="0.3275" h="0.2775" d="0.1525" />
-     </inertial>
+        <mass value="45" />
+        <origin xyz="0.0 0.0 0.0" />
+        <xacro:solid_cuboid_inertia m="45" w="0.3275" h="0.2775" d="0.1525" />
+      </inertial>
       <visual>
         <origin xyz="0 0 0" rpy="0 0 0" />
@@ -42,5 +28,4 @@
         </xacro:if>
         <xacro:unless value="${hq}">
-		  <!-- in this case change origin -->
           <geometry>
             <box size="0.700 0.600 0.350"/>
@@ -54,5 +39,4 @@
         <origin xyz="0 0 0.005" rpy="0 0 0 " />
         <geometry>
-          <!--box size="0.05 0.05 0.01"/-->
           <mesh filename="package://rb_theron_description/meshes/bases/theron_base.dae"/>
         </geometry>

File: rb_theron_description/urdf/common.gazebo.xacro (robot description, xacro)
@@ -1,26 +1,26 @@
 <?xml version="1.0"?>
 <robot xmlns:xacro="http://www.ros.org/wiki/xacro">
-	<!-- ROS CONTROL GAZEBO PLUGIN -->
-	<xacro:macro name="ros_control">
-		<gazebo>
-			<plugin name="ros_control" filename="libgazebo_ros_control.so">
-				<!--robotNamespace>/robot</robotNamespace-->
-				<robotParam>robot/robot_description</robotParam>
-				<controlPeriod>0.001</controlPeriod>
-				<robotSimType>gazebo_ros_control/DefaultRobotHWSim</robotSimType>
-				<legacyModeNS>true</legacyModeNS>
-			</plugin>
-		</gazebo>
-	</xacro:macro>
-	<xacro:macro name="gazebo_colors" params="prefix">
-		<gazebo reference="$(arg prefix)base_footprint">
-			<material>Gazebo/Green</material>
-		</gazebo>
-		<gazebo reference="$(arg prefix)base_link">
-			<material>Gazebo/Grey</material>
-		</gazebo>
-		<gazebo reference="$(arg prefix)front_cover_link">
-			<material>Gazebo/Black</material>
-		</gazebo>
-	</xacro:macro>
+    <!-- ROS CONTROL GAZEBO PLUGIN -->
+    <xacro:macro name="ros_control">
+        <gazebo>
+            <plugin name="ros_control" filename="libgazebo_ros_control.so">
+                <!--robotNamespace>/robot</robotNamespace-->
+                <robotParam>robot/robot_description</robotParam>
+                <controlPeriod>0.001</controlPeriod>
+                <robotSimType>gazebo_ros_control/DefaultRobotHWSim</robotSimType>
+                <legacyModeNS>true</legacyModeNS>
+            </plugin>
+        </gazebo>
+    </xacro:macro>
+    <xacro:macro name="gazebo_colors" params="prefix">
+        <gazebo reference="$(arg prefix)base_footprint">
+            <material>Gazebo/Green</material>
+        </gazebo>
+        <gazebo reference="$(arg prefix)base_link">
+            <material>Gazebo/Grey</material>
+        </gazebo>
+        <gazebo reference="$(arg prefix)front_cover_link">
+            <material>Gazebo/Black</material>
+        </gazebo>
+    </xacro:macro>
 </robot>

File: rb_theron_description/urdf/pole/mcq_pole.urdf.xacro (robot description, xacro)
@@ -1,16 +1,16 @@
 <?xml version="1.0"?>
-<robot name="simple_pole"
-  xmlns:xacro="http://www.ros.org/wiki/xacro">
-	<macro name="box_inertia_robot" params="m x y z">
-	        <inertia  ixx="${m*(y*y+z*z)/12}" ixy = "0" ixz = "0"
-	                  iyy="${m*(x*x+z*z)/12}" iyz = "0"
-	                  izz="${m*(x*x+z*z)/12}" />
-	</macro>
+<robot name="mcq_pole" xmlns:xacro="http://www.ros.org/wiki/xacro">
+  <!-- MACROS -->
+  <macro name="box_inertia_robot" params="m x y z">
+    <inertia ixx="${m*(y*y+z*z)/12}" ixy = "0" ixz = "0"
+             iyy="${m*(x*x+z*z)/12}" iyz = "0"
+             izz="${m*(x*x+z*z)/12}" />
+  </macro>
   <xacro:macro name="mcq_pole" params="prefix parent *origin">
-		<joint name="${prefix}pole_joint" type="fixed">
-			<parent link="${parent}"/>
-			<child link="${prefix}pole_link"/>
-			<xacro:insert_block name="origin" />
-		</joint>
+    <joint name="${prefix}pole_joint" type="fixed">
+      <parent link="${parent}"/>
+      <child link="${prefix}pole_link"/>
+      <xacro:insert_block name="origin" />
+    </joint>
     <!-- BASE_LINK -->
     <link name="${prefix}pole_link">
@@ -18,11 +18,9 @@
         <mass value="10.0" />
         <origin xyz="0 0 0" />
-	    <xacro:box_inertia_robot m="10" x="0.25" y="0.25" z="1.55"/>
+      <xacro:box_inertia_robot m="10" x="0.25" y="0.25" z="1.55"/>
       </inertial>
       <visual>
         <origin xyz="0 0 0" rpy="0 0 0" />
-		  		<!-- in this case change origin -->
           <geometry>
-            <!-- <box size="0.25 0.25 1.55"/> -->
             <mesh filename="package://rb_theron_description/meshes/pole/mcq_pole.stl"/>
           </geometry>
@@ -34,5 +32,4 @@
         <origin xyz="0 0 0" rpy="0 0 0 " />
         <geometry>
-          <!-- <box size="0.25 0.25 1.55"/> -->
           <mesh filename="package://rb_theron_description/meshes/pole/mcq_pole.stl"/>
         </geometry>
@@ -40,25 +37,11 @@
     </link>
     <gazebo reference="${prefix}pole_link">
-			<mu1 value="100.0"/>
-			<mu2 value="100.0"/>
-			<kp value="500000.0" />
-			<kd value="1.0" />
-			<material>Gazebo/Yellow</material>
-			<turnGravityOff>false</turnGravityOff>
-			<!--kp>500000.0</kp>
-			<kd>10.0</kd>
-			<mu1>10</mu1>
-			<mu2>10</mu2>
-			<fdir1>1 0 0</fdir1-->
-			<!--minDepth>0.001</minDepth-->
-			<!--material>Gazebo/Black</material-->
-			<!--mu1 value="10"/>
-			<mu2 value="5"/>
-			<kp value="500000.0" />
-			<kd value="10.0" />
-			<fdir1 value="1 0 0"/>
-			<material>Gazebo/Yellow</material>
-			<turnGravityOff>false</turnGravityOff-->
-		</gazebo>
+      <mu1 value="100.0"/>
+      <mu2 value="100.0"/>
+      <kp value="500000.0" />
+      <kd value="1.0" />
+      <material>Gazebo/Yellow</material>
+      <turnGravityOff>false</turnGravityOff>
+    </gazebo>
   </xacro:macro>
 </robot>

File: rb_theron_description/urdf/pole/simple_pole.urdf.xacro (robot description, xacro)
@@ -1,16 +1,16 @@
 <?xml version="1.0"?>
-<robot name="simple_pole"
-  xmlns:xacro="http://www.ros.org/wiki/xacro">
-	<macro name="box_inertia_robot" params="m x y z">
-	        <inertia  ixx="${m*(y*y+z*z)/12}" ixy = "0" ixz = "0"
-	                  iyy="${m*(x*x+z*z)/12}" iyz = "0"
-	                  izz="${m*(x*x+z*z)/12}" />
-	</macro>
+<robot name="simple_pole" xmlns:xacro="http://www.ros.org/wiki/xacro">
+  <!-- MACROS -->
+  <macro name="box_inertia_robot" params="m x y z">
+    <inertia ixx="${m*(y*y+z*z)/12}" ixy = "0" ixz = "0"
+             iyy="${m*(x*x+z*z)/12}" iyz = "0"
+             izz="${m*(x*x+z*z)/12}" />
+  </macro>
   <xacro:macro name="simple_pole" params="prefix parent *origin">
-		<joint name="${prefix}pole_joint" type="fixed">
-			<parent link="${parent}"/>
-			<child link="${prefix}pole_link"/>
-			<xacro:insert_block name="origin" />
-		</joint>
+    <joint name="${prefix}pole_joint" type="fixed">
+      <parent link="${parent}"/>
+      <child link="${prefix}pole_link"/>
+      <xacro:insert_block name="origin" />
+    </joint>
     <!-- BASE_LINK -->
     <link name="${prefix}pole_link">
@@ -18,11 +18,9 @@
         <mass value="10.0" />
         <origin xyz="0 0 0" />
-	    <xacro:box_inertia_robot m="10" x="0.25" y="0.25" z="1.55"/>
+      <xacro:box_inertia_robot m="10" x="0.25" y="0.25" z="1.55"/>
       </inertial>
       <visual>
         <origin xyz="0 0 0" rpy="0 0 0" />
-		  		<!-- in this case change origin -->
           <geometry>
-            <!-- <box size="0.25 0.25 1.55"/> -->
             <mesh filename="package://rb_theron_description/meshes/pole/simple_pole.dae"/>
           </geometry>
@@ -34,5 +32,4 @@
         <origin xyz="0 0 0" rpy="0 0 0 " />
         <geometry>
-          <!-- <box size="0.25 0.25 1.55"/> -->
           <mesh filename="package://rb_theron_description/meshes/pole/simple_pole.dae"/>
         </geometry>
@@ -40,25 +37,11 @@
     </link>
     <gazebo reference="${prefix}pole_link">
-			<mu1 value="100.0"/>
-			<mu2 value="100.0"/>
-			<kp value="500000.0" />
-			<kd value="1.0" />
-			<material>Gazebo/Yellow</material>
-			<turnGravityOff>false</turnGravityOff>
-			<!--kp>500000.0</kp>
-			<kd>10.0</kd>
-			<mu1>10</mu1>
-			<mu2>10</mu2>
-			<fdir1>1 0 0</fdir1-->
-			<!--minDepth>0.001</minDepth-->
-			<!--material>Gazebo/Black</material-->
-			<!--mu1 value="10"/>
-			<mu2 value="5"/>
-			<kp value="500000.0" />
-			<kd value="10.0" />
-			<fdir1 value="1 0 0"/>
-			<material>Gazebo/Yellow</material>
-			<turnGravityOff>false</turnGravityOff-->
-		</gazebo>
+      <mu1 value="100.0"/>
+      <mu2 value="100.0"/>
+      <kp value="500000.0" />
+      <kd value="1.0" />
+      <material>Gazebo/Yellow</material>
+      <turnGravityOff>false</turnGravityOff>
+    </gazebo>
   </xacro:macro>
 </robot>

File: rb_theron_description/urdf/rocker/mcq_prototype_rocker.urdf.xacro (robot description, xacro)
@@ -14,6 +14,6 @@
   </xacro:macro>
   <xacro:macro name="rocker" params="prefix parent *origin reflect hq">
-	<!--ROCKER BOGIE SUPPORT -->
-	<!--joint name="${prefix}joint_support" type="continuous">
+  <!--ROCKER BOGIE SUPPORT -->
+  <!--joint name="${prefix}joint_support" type="continuous">
       <parent link="${parent}"/>
       <child link="${prefix}support"/>
@@ -22,6 +22,6 @@
       <limit effort="100" velocity="100"/>
       <joint_properties damping="0.1" friction="0.1"/>
-	</joint -->
-	<joint name="${prefix}joint_rsupport" type="revolute">
+  </joint -->
+  <joint name="${prefix}joint_rsupport" type="revolute">
       <parent link="${parent}"/>
       <child link="${prefix}rsupport"/>
@@ -30,11 +30,11 @@
       <limit lower="-0.5" upper="0.5" effort="100" velocity="100"/>
       <joint_properties damping="0.1" friction="0.1"/>
-	</joint>
-	<link name="${prefix}rsupport">
+  </joint>
+  <link name="${prefix}rsupport">
       <visual>
         <origin xyz="0 0 0" rpy="0 0 0" />
           <xacro:if value="${reflect}">
             <geometry>
-	          <mesh filename="package://rb_theron_description/meshes/rocker/mcq_prototype_rocker_r.dae" />
+            <mesh filename="package://rb_theron_description/meshes/rocker/mcq_prototype_rocker_r.dae" />
             </geometry>
           </xacro:if>
@@ -43,5 +43,5 @@
               <mesh filename="package://rb_theron_description/meshes/rocker/mcq_prototype_rocker_l.dae" />
             </geometry>
-		  </xacro:unless>
+      </xacro:unless>
       </visual>
       <collision>
@@ -49,5 +49,5 @@
           <xacro:if value="${reflect}">
             <geometry>
-	          <mesh filename="package://rb_theron_description/meshes/rocker/mcq_prototype_rocker_r.dae" />
+            <mesh filename="package://rb_theron_description/meshes/rocker/mcq_prototype_rocker_r.dae" />
             </geometry>
           </xacro:if>
@@ -56,5 +56,5 @@
               <mesh filename="package://rb_theron_description/meshes/rocker/mcq_prototype_rocker_l.dae" />
             </geometry>
-		  </xacro:unless>
+      </xacro:unless>
       </collision>
       <inertial>
@@ -63,18 +63,18 @@
         <xacro:cylinder_inertia  m="${rocker_support_mass}" r="0.010" h="0.010" />  <!--Check these values -->
       </inertial>
-	</link>
-	<!-- Transmission is important to link the joints and the controller -->
-	<transmission name="${prefix}rsupport_joint_trans">
-	  <type>transmission_interface/SimpleTransmission</type>
-	  <joint name="${prefix}joint_rsupport">
-		  <hardwareInterface>hardware_interface/EffortJointInterface</hardwareInterface>
-	  </joint>
-	  <actuator name="${prefix}rsupport_joint_motor">
-		<mechanicalReduction>1</mechanicalReduction>
-		<motorTorqueConstant>1</motorTorqueConstant>
-	  </actuator>
-	</transmission>
-	<!-- Flag to select the high or low quality model -->
-	<xacro:property name="hq" value="true" />
+  </link>
+  <!-- Transmission is important to link the joints and the controller -->
+  <transmission name="${prefix}rsupport_joint_trans">
+    <type>transmission_interface/SimpleTransmission</type>
+    <joint name="${prefix}joint_rsupport">
+      <hardwareInterface>hardware_interface/EffortJointInterface</hardwareInterface>
+    </joint>
+    <actuator name="${prefix}rsupport_joint_motor">
+    <mechanicalReduction>1</mechanicalReduction>
+    <motorTorqueConstant>1</motorTorqueConstant>
+    </actuator>
+  </transmission>
+  <!-- Flag to select the high or low quality model -->
+  <xacro:property name="hq" value="true" />
     <xacro:property name="wheel_offset_x" value="-0.1175" />
     <xacro:if value="${reflect}">
@@ -82,36 +82,36 @@
     </xacro:if>
     <xacro:unless value="${reflect}">
-		 <xacro:property name="wheel_offset_y" value="0.079" />
+     <xacro:property name="wheel_offset_y" value="0.079" />
     </xacro:unless>
     <xacro:property name="wheel_offset_z" value="-0.0428" />
-	<!-- xacro:rubber_wheel prefix="$(arg prefix)wheel" parent="$(arg prefix)support" reflect="true" hq="${hq}">
-		<origin xyz="${wheel_offset_x} ${wheel_offset_y} ${wheel_offset_z}" rpy="0 0 0"/>
-	</xacro:rubber_wheel -->
-	<xacro:rubber_wheel prefix="${prefix}" parent="${prefix}rsupport" reflect="true" hq="${hq}">
-		<origin xyz="${wheel_offset_x} ${wheel_offset_y} ${wheel_offset_z}" rpy="0 0 0"/>
-	</xacro:rubber_wheel>
+  <!-- xacro:rubber_wheel prefix="$(arg prefix)wheel" parent="$(arg prefix)support" reflect="true" hq="${hq}">
+    <origin xyz="${wheel_offset_x} ${wheel_offset_y} ${wheel_offset_z}" rpy="0 0 0"/>
+  </xacro:rubber_wheel -->
+  <xacro:rubber_wheel prefix="${prefix}" parent="${prefix}rsupport" reflect="true" hq="${hq}">
+    <origin xyz="${wheel_offset_x} ${wheel_offset_y} ${wheel_offset_z}" rpy="0 0 0"/>
+  </xacro:rubber_wheel>
     <xacro:property name="caster_offset_x" value="0.1175" />
     <xacro:property name="caster_offset_y" value="0.010" />
     <xacro:property name="caster_offset_z" value="0.002" />
-	<!-- xacro:caster prefix="$(arg prefix)left" parent="$(arg prefix)support" hq="${hq}">
-		<origin xyz="${caster_offset_x} ${caster_offset_y} ${caster_offset_z}" rpy="0 0 0"/>
-	</xacro:caster -->
-	<xacro:caster prefix="${prefix}castor" parent="${prefix}rsupport" hq="${hq}">
-		<origin xyz="${caster_offset_x} ${caster_offset_y} ${caster_offset_z}" rpy="0 0 0"/>
-	</xacro:caster>
+  <!-- xacro:caster prefix="$(arg prefix)left" parent="$(arg prefix)support" hq="${hq}">
+    <origin xyz="${caster_offset_x} ${caster_offset_y} ${caster_offset_z}" rpy="0 0 0"/>
+  </xacro:caster -->
+  <xacro:caster prefix="${prefix}castor" parent="${prefix}rsupport" hq="${hq}">
+    <origin xyz="${caster_offset_x} ${caster_offset_y} ${caster_offset_z}" rpy="0 0 0"/>
+  </xacro:caster>
     <!-- gazebo reference="${prefix}support">
-			<mu1 value="5.0"/>
-			<mu2 value="0.5"/>
-			<kp value="10000000.0" />
-			<kd value="1.0" />
-			<fdir1 value="1 0 0"/>
+      <mu1 value="5.0"/>
+      <mu2 value="0.5"/>
+      <kp value="10000000.0" />
+      <kd value="1.0" />
+      <fdir1 value="1 0 0"/>
       <turnGravityOff>false</turnGravityOff>
     </gazebo>
      <gazebo reference="${prefix}_wheel">
-			<mu1 value="5.0"/>
-			<mu2 value="0.5"/>
-			<kp value="10000000.0" />
-			<kd value="1.0" />
-			<fdir1 value="1 0 0"/>
+      <mu1 value="5.0"/>
+      <mu2 value="0.5"/>
+      <kp value="10000000.0" />
+      <kd value="1.0" />
+      <fdir1 value="1 0 0"/>
       <turnGravityOff>false</turnGravityOff>
     </gazebo -->

File: rb_theron_description/urdf/wheels/castor.urdf.xacro (robot description, xacro)
@@ -33,5 +33,5 @@
         <origin xyz="0 0 0" rpy="0 0 0" />
           <geometry>
-	       <mesh filename="package://rb_theron_description/meshes/wheels/castor_wheel.stl" />
+         <mesh filename="package://rb_theron_description/meshes/wheels/castor_wheel.stl" />
           </geometry>
       </visual>
@@ -39,5 +39,5 @@
         <origin xyz="0 0 0" rpy="0 0 0" />
           <geometry>
-	       <mesh filename="package://rb_theron_description/meshes/wheels/castor_wheel.dae" />
+         <mesh filename="package://rb_theron_description/meshes/wheels/castor_wheel.dae" />
           </geometry>
       </collision-->
@@ -51,5 +51,5 @@
   <!-- xacro:caster_wheel prefix="${prefix}" parent="${prefix}support" hq="${hq}" -->
   <xacro:caster_wheel prefix="${prefix}" parent="${prefix}support" hq="${hq}">
-		<origin xyz="${caster_wheel_offset_x} ${caster_wheel_offset_y} ${caster_wheel_offset_z}" rpy="0 0 0"/>
+    <origin xyz="${caster_wheel_offset_x} ${caster_wheel_offset_y} ${caster_wheel_offset_z}" rpy="0 0 0"/>
    </xacro:caster_wheel>
  </xacro:macro>
@@ -69,5 +69,5 @@
           <origin xyz="0 0 0" rpy="0 0 0" />
           <geometry>
-		<mesh filename="package://rb_theron_description/meshes/wheels/mcq_prototype_castor_wheel.dae" />
+    <mesh filename="package://rb_theron_description/meshes/wheels/mcq_prototype_castor_wheel.dae" />
           </geometry>
         </xacro:if -->
@@ -82,14 +82,14 @@
       </visual>
      <collision>
-	  <origin xyz="0 0 0" rpy="${M_PI/2} 0 0" />
-	  <!-- origin xyz="0 0 0" rpy="0 0 0" / -->
+    <origin xyz="0 0 0" rpy="${M_PI/2} 0 0" />
+    <!-- origin xyz="0 0 0" rpy="0 0 0" / -->
         <geometry>
-		  <!-- mesh filename="package://rb_theron_description/meshes/wheels/mcq_prototype_castor_wheel.dae" / -->
+      <!-- mesh filename="package://rb_theron_description/meshes/wheels/mcq_prototype_castor_wheel.dae" / -->
           <cylinder length="${caster_height}" radius="${caster_radius}" />
           <!-- sphere radius="${caster_radius}"/ -->
         </geometry>
-		<surface>
+    <surface>
           <bounce restitution_coefficient = "1"/>
-		</surface>
+    </surface>
       </collision>
       <inertial>
@@ -107,5 +107,5 @@
       <actuator name="${prefix}support_joint_motor">
         <mechanicalReduction>1</mechanicalReduction>
-      	<motorTorqueConstant>1</motorTorqueConstant>
+        <motorTorqueConstant>1</motorTorqueConstant>
       </actuator>
     </transmission>
@@ -117,24 +117,24 @@
       <actuator name="${prefix}wheel_joint_motor">
         <mechanicalReduction>1</mechanicalReduction>
-		<motorTorqueConstant>1</motorTorqueConstant>
+    <motorTorqueConstant>1</motorTorqueConstant>
       </actuator>
     </transmission>
     <!-- gazebo reference="${prefix}support">
-			<mu1 value="5.0"/>
-			<mu2 value="0.5"/>
-			<kp value="10000000.0" />
-			<kd value="1.0" />
-			<fdir1 value="1 0 0"/>
+      <mu1 value="5.0"/>
+      <mu2 value="0.5"/>
+      <kp value="10000000.0" />
+      <kd value="1.0" />
+      <fdir1 value="1 0 0"/>
       <turnGravityOff>false</turnGravityOff>
     </gazebo -->
      <gazebo reference="${prefix}_wheel">
-			<mu1 value="100.0"/>
-			<mu2 value="100.0"/>
-			<!-- kp value="10000000.0" / -->
-			<kp value="100000.0" />
-			<kd value="100.0" />
-			<!-- fdir1 value="1 0 0"/ -->
-			<material>Gazebo/Black</material>
-			<turnGravityOff>false</turnGravityOff>
+      <mu1 value="100.0"/>
+      <mu2 value="100.0"/>
+      <!-- kp value="10000000.0" / -->
+      <kp value="100000.0" />
+      <kd value="100.0" />
+      <!-- fdir1 value="1 0 0"/ -->
+      <material>Gazebo/Black</material>
+      <turnGravityOff>false</turnGravityOff>
     </gazebo>
  </xacro:macro>
