Commit message: Changed tabs to spaces and removed spaces

File: rb_theron_description/urdf/wheels/rubber_wheel.gazebo.xacro (robot description, xacro)
@@ -1,54 +1,54 @@
 <?xml version="1.0"?>
 <robot xmlns:xacro="http://www.ros.org/wiki/xacro">
-	<xacro:macro name="rubber_wheel_gazebo" params="prefix">
-		<gazebo reference="${prefix}_wheel_link">
-			<!-- mu1 value="5.0"/>
-			<mu2 value="0.5"/>
-			<kp value="10000000.0" />
-			<kd value="1.0" />
-			<fdir1 value="1 0 0"/>
-			<material>Gazebo/Yellow</material>
-			<turnGravityOff>false</turnGravityOff -->
-			<!-- mu1 value="5.0"/>
-			<mu2 value="0.5"/ -->
-			<mu1 value="100.0"/>
-			<mu2 value="100.0"/>
-			<!-- kp value="100000.0" / -->
-			<kp value="500000.0" />
-			<kd value="1.0" />
-			<!-- fdir1 value="1 0 0"/ -->
-			<material>Gazebo/Yellow</material>
-			<turnGravityOff>false</turnGravityOff>
-			<!--kp>500000.0</kp>
-			<kd>10.0</kd>
-			<mu1>10</mu1>
-			<mu2>10</mu2>
-			<fdir1>1 0 0</fdir1-->
-			<!--minDepth>0.001</minDepth-->
-			<!--material>Gazebo/Black</material-->
-			<!--mu1 value="10"/>
-			<mu2 value="5"/>
-			<kp value="500000.0" />
-			<kd value="10.0" />
-			<fdir1 value="1 0 0"/>
-			<material>Gazebo/Yellow</material>
-			<turnGravityOff>false</turnGravityOff-->
-		</gazebo>
-		<gazebo reference="${prefix}_wheel_tire_link">
-			<material>Gazebo/Gray</material>
-			<turnGravityOff>false</turnGravityOff>
-		</gazebo>
-		<!--gazebo reference="${name}_wheel_link">
-			<kp>500000.0</kp>
-			<kd>10.0</kd>
-			<mu1>10</mu1>
-			<mu2>10</mu2>
-			<fdir1>1 0 0</fdir1>
-			<maxVel>1.0</maxVel>
-			<minDepth>0.003</minDepth>
-			<material>Gazebo/Yellow</material>
-			<turnGravityOff>false</turnGravityOff>
-			<implicitSpringDamper>1</implicitSpringDamper>
-		</gazebo-->
-	</xacro:macro>
+    <xacro:macro name="rubber_wheel_gazebo" params="prefix">
+        <gazebo reference="${prefix}_wheel_link">
+            <!-- mu1 value="5.0"/>
+            <mu2 value="0.5"/>
+            <kp value="10000000.0" />
+            <kd value="1.0" />
+            <fdir1 value="1 0 0"/>
+            <material>Gazebo/Yellow</material>
+            <turnGravityOff>false</turnGravityOff -->
+            <!-- mu1 value="5.0"/>
+            <mu2 value="0.5"/ -->
+            <mu1 value="100.0"/>
+            <mu2 value="100.0"/>
+            <!-- kp value="100000.0" / -->
+            <kp value="500000.0" />
+            <kd value="1.0" />
+            <!-- fdir1 value="1 0 0"/ -->
+            <material>Gazebo/Yellow</material>
+            <turnGravityOff>false</turnGravityOff>
+            <!--kp>500000.0</kp>
+            <kd>10.0</kd>
+            <mu1>10</mu1>
+            <mu2>10</mu2>
+            <fdir1>1 0 0</fdir1-->
+            <!--minDepth>0.001</minDepth-->
+            <!--material>Gazebo/Black</material-->
+            <!--mu1 value="10"/>
+            <mu2 value="5"/>
+            <kp value="500000.0" />
+            <kd value="10.0" />
+            <fdir1 value="1 0 0"/>
+            <material>Gazebo/Yellow</material>
+            <turnGravityOff>false</turnGravityOff-->
+        </gazebo>
+        <gazebo reference="${prefix}_wheel_tire_link">
+            <material>Gazebo/Gray</material>
+            <turnGravityOff>false</turnGravityOff>
+        </gazebo>
+        <!--gazebo reference="${name}_wheel_link">
+            <kp>500000.0</kp>
+            <kd>10.0</kd>
+            <mu1>10</mu1>
+            <mu2>10</mu2>
+            <fdir1>1 0 0</fdir1>
+            <maxVel>1.0</maxVel>
+            <minDepth>0.003</minDepth>
+            <material>Gazebo/Yellow</material>
+            <turnGravityOff>false</turnGravityOff>
+            <implicitSpringDamper>1</implicitSpringDamper>
+        </gazebo-->
+    </xacro:macro>
 </robot>

File: rb_theron_description/urdf/wheels/rubber_wheel.transmission.xacro (robot description, xacro)
@@ -1,20 +1,20 @@
 <?xml version="1.0"?>
 <robot xmlns:xacro="http://www.ros.org/wiki/xacro">
-	<!-- Rubber wheel transmission -->
-	<xacro:macro name="rubber_wheel_transmission" params="prefix">
-	<!-- Transmission is important to link the joints and the controller (see rb_theron_control/config/rb_theron_control.yaml)-->
-		<transmission name="${prefix}_wheel_joint_trans">
-			<type>transmission_interface/SimpleTransmission</type>
-			<joint name="${prefix}_wheel_joint">
-				<!-- for the gazebo plugin -->
-				<!--hardwareInterface>EffortJointInterface</hardwareInterface-->
-				<!-- for ros control controller -->
-				<hardwareInterface>hardware_interface/VelocityJointInterface</hardwareInterface>
-			</joint>
-			<actuator name="${prefix}_wheel_joint_motor">
-				<mechanicalReduction>1</mechanicalReduction>
-				<motorTorqueConstant>20</motorTorqueConstant>
-			</actuator>
-		</transmission>
-	</xacro:macro>
+    <!-- Rubber wheel transmission -->
+    <xacro:macro name="rubber_wheel_transmission" params="prefix">
+    <!-- Transmission is important to link the joints and the controller (see rb_theron_control/config/rb_theron_control.yaml)-->
+        <transmission name="${prefix}_wheel_joint_trans">
+            <type>transmission_interface/SimpleTransmission</type>
+            <joint name="${prefix}_wheel_joint">
+                <!-- for the gazebo plugin -->
+                <!--hardwareInterface>EffortJointInterface</hardwareInterface-->
+                <!-- for ros control controller -->
+                <hardwareInterface>hardware_interface/VelocityJointInterface</hardwareInterface>
+            </joint>
+            <actuator name="${prefix}_wheel_joint_motor">
+                <mechanicalReduction>1</mechanicalReduction>
+                <motorTorqueConstant>20</motorTorqueConstant>
+            </actuator>
+        </transmission>
+    </xacro:macro>
 </robot>

File: rb_theron_description/urdf/wheels/rubber_wheel.urdf.xacro (robot description, xacro)
@@ -1,49 +1,49 @@
 <?xml version="1.0"?>
 <robot name="wheel"
-	xmlns:xacro="http://www.ros.org/wiki/xacro">
-	<xacro:include filename="$(find rb_theron_description)/urdf/wheels/rubber_wheel.transmission.xacro"/>
-	<xacro:include filename="$(find rb_theron_description)/urdf/wheels/rubber_wheel.gazebo.xacro"/>
-	<xacro:property name="M_PI" value="3.1415926535897931" />
-	<!-- Wheels -->
-	<xacro:property name="wheel_radius" value="0.125" />
-	<xacro:property name="wheel_height" value="0.032" />
-	<xacro:property name="wheel_mass" value="1.0" />
-	<!-- in kg-->
-	<xacro:macro name="cylinder_inertia" params="m r h">
-		<inertia ixx="${m*(3*r*r+h*h)/12}" ixy = "0" ixz = "0" iyy="${m*(3*r*r+h*h)/12}" iyz = "0" izz="${m*r*r/2}" />
-	</xacro:macro>
-	<xacro:macro name="rubber_wheel" params="prefix parent *origin reflect hq">
-		<!--WHEEL TIRE -->
-		<joint name="${prefix}_wheel_joint" type="continuous">
-			<parent link="${parent}"/>
-			<child link="${prefix}_wheel_link"/>
-			<xacro:insert_block name="origin" />
-			<axis xyz="0 1 0" rpy="0 0 0" />
-			<limit effort="100" velocity="100"/>
-			<joint_properties damping="0.0" friction="0.0"/>
-		</joint>
-		<link name="${prefix}_wheel_link">
-			<visual>
-				<!-- HIGH RESOLUTION WHEELS -->
-				<!-- LOW RESOLUTION WHEELS -->
-				<origin xyz="0 0 0" rpy="${M_PI/2} 0 0" />
-				<geometry>
-					<cylinder length="${wheel_height}" radius="${wheel_radius}" />
-				</geometry>
-			</visual>
-			<collision>
-				<origin xyz="0 0 0" rpy="${M_PI/2} 0 0" />
-				<geometry>
-					<cylinder length="${wheel_height}" radius="${wheel_radius}" />
-				</geometry>
-			</collision>
-			<inertial>
-				<mass value="${wheel_mass}" />
-				<origin xyz="0 0 0" />
-				<cylinder_inertia m="${wheel_mass}" r="${wheel_radius}" h="${wheel_height}" />
-			</inertial>
-		</link>
-		<xacro:rubber_wheel_transmission prefix="${prefix}" />
-		<xacro:rubber_wheel_gazebo prefix="${prefix}" />
-	</xacro:macro>
+    xmlns:xacro="http://www.ros.org/wiki/xacro">
+    <xacro:include filename="$(find rb_theron_description)/urdf/wheels/rubber_wheel.transmission.xacro"/>
+    <xacro:include filename="$(find rb_theron_description)/urdf/wheels/rubber_wheel.gazebo.xacro"/>
+    <xacro:property name="M_PI" value="3.1415926535897931" />
+    <!-- Wheels -->
+    <xacro:property name="wheel_radius" value="0.125" />
+    <xacro:property name="wheel_height" value="0.032" />
+    <xacro:property name="wheel_mass" value="1.0" />
+    <!-- in kg-->
+    <xacro:macro name="cylinder_inertia" params="m r h">
+        <inertia ixx="${m*(3*r*r+h*h)/12}" ixy = "0" ixz = "0" iyy="${m*(3*r*r+h*h)/12}" iyz = "0" izz="${m*r*r/2}" />
+    </xacro:macro>
+    <xacro:macro name="rubber_wheel" params="prefix parent *origin reflect hq">
+        <!--WHEEL TIRE -->
+        <joint name="${prefix}_wheel_joint" type="continuous">
+            <parent link="${parent}"/>
+            <child link="${prefix}_wheel_link"/>
+            <xacro:insert_block name="origin" />
+            <axis xyz="0 1 0" rpy="0 0 0" />
+            <limit effort="100" velocity="100"/>
+            <joint_properties damping="0.0" friction="0.0"/>
+        </joint>
+        <link name="${prefix}_wheel_link">
+            <visual>
+                <!-- HIGH RESOLUTION WHEELS -->
+                <!-- LOW RESOLUTION WHEELS -->
+                <origin xyz="0 0 0" rpy="${M_PI/2} 0 0" />
+                <geometry>
+                    <cylinder length="${wheel_height}" radius="${wheel_radius}" />
+                </geometry>
+            </visual>
+            <collision>
+                <origin xyz="0 0 0" rpy="${M_PI/2} 0 0" />
+                <geometry>
+                    <cylinder length="${wheel_height}" radius="${wheel_radius}" />
+                </geometry>
+            </collision>
+            <inertial>
+                <mass value="${wheel_mass}" />
+                <origin xyz="0 0 0" />
+                <cylinder_inertia m="${wheel_mass}" r="${wheel_radius}" h="${wheel_height}" />
+            </inertial>
+        </link>
+        <xacro:rubber_wheel_transmission prefix="${prefix}" />
+        <xacro:rubber_wheel_gazebo prefix="${prefix}" />
+    </xacro:macro>
 </robot>

File: rb_theron_description/urdf/wheels/rubber_wheel_125.urdf.xacro (robot description, xacro)
@@ -1,49 +1,48 @@
 <?xml version="1.0"?>
-<robot name="wheel"
-	xmlns:xacro="http://www.ros.org/wiki/xacro">
-	<xacro:include filename="$(find rb_theron_description)/urdf/wheels/rubber_wheel.transmission.xacro"/>
-	<xacro:include filename="$(find rb_theron_description)/urdf/wheels/rubber_wheel.gazebo.xacro"/>
-	<xacro:property name="M_PI" value="3.1415926535897931" />
-	<!-- Wheels -->
-	<xacro:property name="wheel_radius" value="0.0762" />
-	<xacro:property name="wheel_height" value="0.032" />
-	<xacro:property name="wheel_mass" value="0.25" />
-	<!-- in kg-->
-	<xacro:macro name="cylinder_inertia" params="m r h">
-		<inertia ixx="${m*(3*r*r+h*h)/12}" ixy = "0" ixz = "0" iyy="${m*(3*r*r+h*h)/12}" iyz = "0" izz="${m*r*r/2}" />
-	</xacro:macro>
-	<xacro:macro name="rubber_wheel" params="prefix parent *origin reflect hq">
-		<!--WHEEL TIRE -->
-		<joint name="${prefix}_wheel_joint" type="continuous">
-			<parent link="${parent}"/>
-			<child link="${prefix}_wheel_link"/>
-			<xacro:insert_block name="origin" />
-			<axis xyz="0 1 0" rpy="0 0 0" />
-			<limit effort="100" velocity="100"/>
-			<joint_properties damping="0.0" friction="0.0"/>
-		</joint>
-		<link name="${prefix}_wheel_link">
-			<visual>
-				<!-- HIGH RESOLUTION WHEELS -->
-				<!-- LOW RESOLUTION WHEELS -->
-				<origin xyz="0 0 0" rpy="${M_PI/2} 0 0" />
-				<geometry>
-					<cylinder length="${wheel_height}" radius="${wheel_radius}" />
-				</geometry>
-			</visual>
-			<collision>
-				<origin xyz="0 0 0" rpy="${M_PI/2} 0 0" />
-				<geometry>
-					<cylinder length="${wheel_height}" radius="${wheel_radius}" />
-				</geometry>
-			</collision>
-			<inertial>
-				<mass value="${wheel_mass}" />
-				<origin xyz="0 0 0" />
-				<cylinder_inertia m="${wheel_mass}" r="${wheel_radius}" h="${wheel_height}" />
-			</inertial>
-		</link>
-		<xacro:rubber_wheel_transmission prefix="${prefix}" />
-		<xacro:rubber_wheel_gazebo prefix="${prefix}" />
-	</xacro:macro>
+<robot name="wheel" xmlns:xacro="http://www.ros.org/wiki/xacro">
+    <xacro:include filename="$(find rb_theron_description)/urdf/wheels/rubber_wheel.transmission.xacro"/>
+    <xacro:include filename="$(find rb_theron_description)/urdf/wheels/rubber_wheel.gazebo.xacro"/>
+    <xacro:property name="M_PI" value="3.1415926535897931" />
+    <!-- Wheels -->
+    <xacro:property name="wheel_radius" value="0.0762" />
+    <xacro:property name="wheel_height" value="0.032" />
+    <xacro:property name="wheel_mass" value="0.25" />
+    <!-- in kg-->
+    <xacro:macro name="cylinder_inertia" params="m r h">
+        <inertia ixx="${m*(3*r*r+h*h)/12}" ixy = "0" ixz = "0" iyy="${m*(3*r*r+h*h)/12}" iyz = "0" izz="${m*r*r/2}" />
+    </xacro:macro>
+    <xacro:macro name="rubber_wheel" params="prefix parent *origin reflect hq">
+        <!--WHEEL TIRE -->
+        <joint name="${prefix}_wheel_joint" type="continuous">
+            <parent link="${parent}"/>
+            <child link="${prefix}_wheel_link"/>
+            <xacro:insert_block name="origin" />
+            <axis xyz="0 1 0" rpy="0 0 0" />
+            <limit effort="100" velocity="100"/>
+            <joint_properties damping="0.0" friction="0.0"/>
+        </joint>
+        <link name="${prefix}_wheel_link">
+            <visual>
+                <!-- HIGH RESOLUTION WHEELS -->
+                <!-- LOW RESOLUTION WHEELS -->
+                <origin xyz="0 0 0" rpy="${M_PI/2} 0 0" />
+                <geometry>
+                    <cylinder length="${wheel_height}" radius="${wheel_radius}" />
+                </geometry>
+            </visual>
+            <collision>
+                <origin xyz="0 0 0" rpy="${M_PI/2} 0 0" />
+                <geometry>
+                    <cylinder length="${wheel_height}" radius="${wheel_radius}" />
+                </geometry>
+            </collision>
+            <inertial>
+                <mass value="${wheel_mass}" />
+                <origin xyz="0 0 0" />
+                <cylinder_inertia m="${wheel_mass}" r="${wheel_radius}" h="${wheel_height}" />
+            </inertial>
+        </link>
+        <xacro:rubber_wheel_transmission prefix="${prefix}" />
+        <xacro:rubber_wheel_gazebo prefix="${prefix}" />
+    </xacro:macro>
 </robot>

File: rb_theron_description/urdf/wheels/rubber_wheel_150.urdf.xacro (robot description, xacro)
@@ -1,62 +1,62 @@
 <?xml version="1.0"?>
 <robot name="wheel"
-	xmlns:xacro="http://www.ros.org/wiki/xacro">
-	<xacro:include filename="$(find rb_theron_description)/urdf/wheels/rubber_wheel.transmission.xacro"/>
-	<xacro:include filename="$(find rb_theron_description)/urdf/wheels/rubber_wheel.gazebo.xacro"/>
-	<xacro:property name="M_PI" value="3.1415926535897931" />
-	<!-- Wheels -->
-	<xacro:property name="wheel_radius" value="0.0756" />
-	<xacro:property name="wheel_height" value="0.025" />
-	<xacro:property name="wheel_mass" value="1" />
-	<!-- in kg-->
-	<xacro:macro name="cylinder_inertia" params="m r h">
-		<inertia ixx="${m*(3*r*r+h*h)/12}" ixy = "0" ixz = "0" iyy="${m*(3*r*r+h*h)/12}" iyz = "0" izz="${m*r*r/2}" />
-	</xacro:macro>
-	<xacro:macro name="rubber_wheel" params="prefix parent *origin hq">
-		<!--WHEEL TIRE -->
-		<joint name="${prefix}_wheel_joint" type="continuous">
-			<parent link="${parent}"/>
-			<child link="${prefix}_wheel_link"/>
-			<xacro:insert_block name="origin" />
-			<axis xyz="0 1 0" rpy="0 0 0" />
-			<limit effort="100" velocity="100"/>
-			<joint_properties damping="0.0" friction="0.0"/>
-		</joint>
-		<link name="${prefix}_wheel_link">
-			<visual>
-				<!-- HIGH RESOLUTION WHEELS -->
-				<!-- LOW RESOLUTION WHEELS -->
-				<origin xyz="0 0 0" rpy="${M_PI/2} 0 0" />
-				<geometry>
-					<cylinder length="${wheel_height}" radius="${wheel_radius}" />
-				</geometry>
-			</visual>
-			<collision>
-				<origin xyz="0 0 0" rpy="${M_PI/2} 0 0" />
-				<geometry>
-					<cylinder length="${wheel_height}" radius="${wheel_radius}" />
-				</geometry>
-			</collision>
-			<inertial>
-				<mass value="${wheel_mass}" />
-				<origin xyz="0 0 0" />
-				<xacro:cylinder_inertia m="${wheel_mass}" r="${wheel_radius}" h="${wheel_height}" />
-			</inertial>
-		</link>
-		<joint name="${prefix}_wheel_tire_joint" type="fixed">
-			<parent link="${prefix}_wheel_link"/>
-			<child link="${prefix}_wheel_tire_link"/>
-			<origin xyz="0 0 0" rpy="0 0 0" />
-		</joint>
-		<link name="${prefix}_wheel_tire_link">
-			<visual>
+    xmlns:xacro="http://www.ros.org/wiki/xacro">
+    <xacro:include filename="$(find rb_theron_description)/urdf/wheels/rubber_wheel.transmission.xacro"/>
+    <xacro:include filename="$(find rb_theron_description)/urdf/wheels/rubber_wheel.gazebo.xacro"/>
+    <xacro:property name="M_PI" value="3.1415926535897931" />
+    <!-- Wheels -->
+    <xacro:property name="wheel_radius" value="0.0756" />
+    <xacro:property name="wheel_height" value="0.025" />
+    <xacro:property name="wheel_mass" value="1" />
+    <!-- in kg-->
+    <xacro:macro name="cylinder_inertia" params="m r h">
+        <inertia ixx="${m*(3*r*r+h*h)/12}" ixy = "0" ixz = "0" iyy="${m*(3*r*r+h*h)/12}" iyz = "0" izz="${m*r*r/2}" />
+    </xacro:macro>
+    <xacro:macro name="rubber_wheel" params="prefix parent *origin hq">
+        <!--WHEEL TIRE -->
+        <joint name="${prefix}_wheel_joint" type="continuous">
+            <parent link="${parent}"/>
+            <child link="${prefix}_wheel_link"/>
+            <xacro:insert_block name="origin" />
+            <axis xyz="0 1 0" rpy="0 0 0" />
+            <limit effort="100" velocity="100"/>
+            <joint_properties damping="0.0" friction="0.0"/>
+        </joint>
+        <link name="${prefix}_wheel_link">
+            <visual>
+                <!-- HIGH RESOLUTION WHEELS -->
+                <!-- LOW RESOLUTION WHEELS -->
+                <origin xyz="0 0 0" rpy="${M_PI/2} 0 0" />
+                <geometry>
+                    <cylinder length="${wheel_height}" radius="${wheel_radius}" />
+                </geometry>
+            </visual>
+            <collision>
+                <origin xyz="0 0 0" rpy="${M_PI/2} 0 0" />
+                <geometry>
+                    <cylinder length="${wheel_height}" radius="${wheel_radius}" />
+                </geometry>
+            </collision>
+            <inertial>
+                <mass value="${wheel_mass}" />
+                <origin xyz="0 0 0" />
+                <xacro:cylinder_inertia m="${wheel_mass}" r="${wheel_radius}" h="${wheel_height}" />
+            </inertial>
+        </link>
+        <joint name="${prefix}_wheel_tire_joint" type="fixed">
+            <parent link="${prefix}_wheel_link"/>
+            <child link="${prefix}_wheel_tire_link"/>
+            <origin xyz="0 0 0" rpy="0 0 0" />
+        </joint>
+        <link name="${prefix}_wheel_tire_link">
+            <visual>
         <origin xyz="0 0 0" rpy="${M_PI/2} 0 0" />
-				<geometry>
-					<cylinder length="${wheel_height + 0.001}" radius="${wheel_radius * 0.92}" />
-				</geometry>
-			</visual>
-		</link>
-		<xacro:rubber_wheel_transmission prefix="${prefix}" />
-		<xacro:rubber_wheel_gazebo prefix="${prefix}" />
-	</xacro:macro>
+                <geometry>
+                    <cylinder length="${wheel_height + 0.001}" radius="${wheel_radius * 0.92}" />
+                </geometry>
+            </visual>
+        </link>
+        <xacro:rubber_wheel_transmission prefix="${prefix}" />
+        <xacro:rubber_wheel_gazebo prefix="${prefix}" />
+    </xacro:macro>
 </robot>
