Commit message: Restore package://

File: rb_theron_description/urdf/bases/theron_base.urdf.xacro (robot description, xacro)
@@ -24,5 +24,5 @@
         <xacro:if value="${hq}">
           <geometry>
-            <mesh filename="file://$(find rb_theron_description)/meshes/bases/theron_base.stl"/>
+            <mesh filename="package://rb_theron_description/meshes/bases/theron_base.stl"/>
           </geometry>
         </xacro:if>
@@ -39,5 +39,5 @@
         <origin xyz="0 0 0.005" rpy="0 0 0 " />
         <geometry>
-          <mesh filename="file://$(find rb_theron_description)/meshes/bases/theron_base.dae"/>
+          <mesh filename="package://rb_theron_description/meshes/bases/theron_base.dae"/>
         </geometry>
       </collision>

File: rb_theron_description/urdf/pole/mcq_pole.urdf.xacro (robot description, xacro)
@@ -23,5 +23,5 @@
         <origin xyz="0 0 0" rpy="0 0 0" />
           <geometry>
-            <mesh filename="file://$(find rb_theron_description)/meshes/pole/mcq_pole.stl"/>
+            <mesh filename="package://rb_theron_description/meshes/pole/mcq_pole.stl"/>
           </geometry>
         <material name="darkgrey">
@@ -32,5 +32,5 @@
         <origin xyz="0 0 0" rpy="0 0 0 " />
         <geometry>
-          <mesh filename="file://$(find rb_theron_description)/meshes/pole/mcq_pole.stl"/>
+          <mesh filename="package://rb_theron_description/meshes/pole/mcq_pole.stl"/>
         </geometry>
       </collision>

File: rb_theron_description/urdf/pole/simple_pole.urdf.xacro (robot description, xacro)
@@ -23,5 +23,5 @@
         <origin xyz="0 0 0" rpy="0 0 0" />
           <geometry>
-            <mesh filename="file://$(find rb_theron_description)/meshes/pole/simple_pole.dae"/>
+            <mesh filename="package://rb_theron_description/meshes/pole/simple_pole.dae"/>
           </geometry>
         <material name="darkgrey">
@@ -32,5 +32,5 @@
         <origin xyz="0 0 0" rpy="0 0 0 " />
         <geometry>
-          <mesh filename="file://$(find rb_theron_description)/meshes/pole/simple_pole.dae"/>
+          <mesh filename="package://rb_theron_description/meshes/pole/simple_pole.dae"/>
         </geometry>
       </collision>

File: rb_theron_description/urdf/rocker/mcq_prototype_rocker.urdf.xacro (robot description, xacro)
@@ -36,10 +36,10 @@
           <xacro:if value="${reflect}">
             <geometry>
-            <mesh filename="file://$(find rb_theron_description)/meshes/rocker/mcq_prototype_rocker_r.dae" />
+            <mesh filename="package://rb_theron_description/meshes/rocker/mcq_prototype_rocker_r.dae" />
             </geometry>
           </xacro:if>
           <xacro:unless value="${reflect}">
             <geometry>
-              <mesh filename="file://$(find rb_theron_description)/meshes/rocker/mcq_prototype_rocker_l.dae" />
+              <mesh filename="package://rb_theron_description/meshes/rocker/mcq_prototype_rocker_l.dae" />
             </geometry>
       </xacro:unless>
@@ -49,10 +49,10 @@
           <xacro:if value="${reflect}">
             <geometry>
-            <mesh filename="file://$(find rb_theron_description)/meshes/rocker/mcq_prototype_rocker_r.dae" />
+            <mesh filename="package://rb_theron_description/meshes/rocker/mcq_prototype_rocker_r.dae" />
             </geometry>
           </xacro:if>
           <xacro:unless value="${reflect}">
             <geometry>
-              <mesh filename="file://$(find rb_theron_description)/meshes/rocker/mcq_prototype_rocker_l.dae" />
+              <mesh filename="package://rb_theron_description/meshes/rocker/mcq_prototype_rocker_l.dae" />
             </geometry>
       </xacro:unless>

File: rb_theron_description/urdf/wheels/castor.urdf.xacro (robot description, xacro)
@@ -29,5 +29,5 @@
         <origin xyz="0 0 0" rpy="0 0 0" />
           <geometry>
-         <mesh filename="file://$(find rb_theron_description)/meshes/wheels/castor_wheel.stl" />
+         <mesh filename="package://rb_theron_description/meshes/wheels/castor_wheel.stl" />
           </geometry>
       </visual>

Commit message: description: Fix cylinder_inertia xacro tag

File: rb_theron_description/urdf/bases/theron_base.urdf.xacro (robot description, xacro)
@@ -2,9 +2,9 @@
 <robot name="rbogie_base"
   xmlns:xacro="http://www.ros.org/wiki/xacro">
-<!--macro name="box_inertia_robot" params="m x y z">
+<xacro:macro name="box_inertia_robot" params="m x y z">
         <inertia  ixx="${m*(y*y+z*z)/12}" ixy = "0" ixz = "0"
                   iyy="${m*(x*x+z*z)/12}" iyz = "0"
                   izz="${m*(x*x+z*z)/12}" />
-</macro-->
+</xacro:macro>
   <xacro:macro name="theron_base" params="prefix publish_bf hq">
     <!-- Robot mechanical and motor parameters -->
