Commit message: Update inertias in rb_theron wheels for better performance

File: rb_theron_description/urdf/wheels/rubber_wheel.gazebo.xacro (robot description, xacro)
@@ -12,8 +12,8 @@
 			<!-- mu1 value="5.0"/>
 			<mu2 value="0.5"/ -->
-			<mu1 value="100.0"/>
-			<mu2 value="100.0"/>
+			<mu1 value="1.0"/>
+			<mu2 value="1.0"/>
 			<!-- kp value="100000.0" / -->
-			<kp value="500000.0" />
+			<kp value="10000000.0" />
 			<kd value="1.0" />
 			<!-- fdir1 value="1 0 0"/ -->

File: rb_theron_description/urdf/wheels/rubber_wheel_150.urdf.xacro (robot description, xacro)
@@ -6,11 +6,13 @@
 	<xacro:property name="M_PI" value="3.1415926535897931" />
 	<!-- Wheels -->
-	<xacro:property name="wheel_radius" value="0.0756" />
+	<xacro:property name="wheel_radius" value="0.0762" />
 	<xacro:property name="wheel_height" value="0.025" />
 	<xacro:property name="wheel_mass" value="1" />
 	<!-- in kg-->
 	<xacro:macro name="cylinder_inertia" params="m r h">
-		<inertia ixx="${m*(3*r*r+h*h)/12}" ixy = "0" ixz = "0" iyy="${m*(3*r*r+h*h)/12}" iyz = "0" izz="${m*r*r/2}" />
-	</xacro:macro>
+		<inertia  ixx="${m*(3*r*r+h*h)/12}" ixy = "0" ixz = "0"
+				  iyy="${m*r*r/2}" iyz = "0"
+				  izz="${m*(3*r*r+h*h)/12}" />
+	  </xacro:macro>
 	<xacro:macro name="rubber_wheel" params="prefix parent *origin hq">
 		<!--WHEEL TIRE -->
@@ -40,5 +42,5 @@
 			<inertial>
 				<mass value="${wheel_mass}" />
-				<origin xyz="0 0 0" />
+				<origin xyz="0 0 0" rpy="${M_PI} 0 0" />
 				<xacro:cylinder_inertia m="${wheel_mass}" r="${wheel_radius}" h="${wheel_height}" />
 			</inertial>
