Commit message: rb_theron_description: Update rubber_wheel_140.urdf.xacro to use zltech wheel stl

File: rb_theron_description/urdf/wheels/rubber_wheel_140.urdf.xacro (robot description, xacro)
@@ -13,5 +13,5 @@
 		<inertia ixx="${m*(3*r*r+h*h)/12}" ixy = "0" ixz = "0" iyy="${m*(3*r*r+h*h)/12}" iyz = "0" izz="${m*r*r/2}" />
 	</xacro:macro>
-	<xacro:macro name="rubber_wheel" params="prefix parent *origin hq">
+	<xacro:macro name="rubber_wheel" params="prefix parent reflect *origin hq">
 		<!--WHEEL TIRE -->
 		<joint name="${prefix}_wheel_joint" type="continuous">
@@ -27,13 +27,24 @@
 				<!-- HIGH RESOLUTION WHEELS -->
 				<!-- LOW RESOLUTION WHEELS -->
-				<origin xyz="0 0 0" rpy="${M_PI/2} 0 0" />
+				<xacro:unless value="${reflect}">
+					<origin xyz="0 0 0" rpy="${M_PI} 0 ${M_PI/2}" />
+				</xacro:unless>
+				<xacro:if value="${reflect}">
+					<origin xyz="0 0 0" rpy="${M_PI} 0 ${-M_PI/2}" />
+				</xacro:if>
 				<geometry>
-					<cylinder length="${wheel_height}" radius="${wheel_radius}" />
+					<!-- <cylinder length="${wheel_height}" radius="${wheel_radius}" /> -->
+					<mesh filename="package://rb_theron_description/meshes/wheels/rubber_wheel_zltech.stl" />
 				</geometry>
 			</visual>
 			<collision>
-				<origin xyz="0 0 0" rpy="${M_PI/2} 0 0" />
+				<xacro:unless value="${reflect}">
+					<origin xyz="0 0 0" rpy="${M_PI} 0 ${M_PI/2}" />
+				</xacro:unless>
+				<xacro:if value="${reflect}">
+					<origin xyz="0 0 0" rpy="${M_PI} 0 ${-M_PI/2}" />
+				</xacro:if>
 				<geometry>
-					<cylinder length="${wheel_height}" radius="${wheel_radius}" />
+					<mesh filename="package://rb_theron_description/meshes/wheels/rubber_wheel_zltech.stl" />
 				</geometry>
 			</collision>
@@ -44,5 +55,5 @@
 			</inertial>
 		</link>
-		<joint name="${prefix}_wheel_tire_joint" type="fixed">
+		<!-- <joint name="${prefix}_wheel_tire_joint" type="fixed">
 			<parent link="${prefix}_wheel_link"/>
 			<child link="${prefix}_wheel_tire_link"/>
@@ -56,5 +67,5 @@
 				</geometry>
 			</visual>
-		</link>
+		</link> -->
 		<xacro:rubber_wheel_transmission prefix="${prefix}" />
 		<xacro:rubber_wheel_gazebo prefix="${prefix}" />
