Commit message: Fixed urdf issues

File: rb_theron_description/urdf/wheels/castor.urdf.xacro (robot description, xacro)
@@ -3,9 +3,9 @@
   <xacro:property name="M_PI" value="3.1415926535897931" />
   <!-- Caster support parameters -->
-  <property name="caster_support_mass" value="1.5" /> <!-- in kg-->
+  <xacro:property name="caster_support_mass" value="1.5" /> <!-- in kg-->
   <!-- Caster wheel parameters -->
-  <property name="caster_radius" value="0.050" />
-  <property name="caster_height" value="0.025" />
-  <property name="caster_mass" value="0.25" /> <!-- in kg-->
+  <xacro:property name="caster_radius" value="0.050" />
+  <xacro:property name="caster_height" value="0.025" />
+  <xacro:property name="caster_mass" value="0.25" /> <!-- in kg-->
   <!-- Caster wheel offset-->
   <xacro:property name="caster_wheel_offset_x" value="-0.033" />
@@ -45,5 +45,5 @@
         <mass value="${caster_support_mass}" />
         <origin xyz="0 0 0" />
-        <cylinder_inertia  m="${caster_support_mass}" r="0.010" h="0.010" />  <!--Check these values -->
+        <xacro:cylinder_inertia  m="${caster_support_mass}" r="0.010" h="0.010" />  <!--Check these values -->
       </inertial>
     </link>
@@ -96,5 +96,5 @@
         <mass value="${caster_mass}" />
         <origin xyz="0 0 0" />
-        <cylinder_inertia  m="${caster_mass}" r="${caster_radius}" h="${caster_height}" />
+        <xacro:cylinder_inertia  m="${caster_mass}" r="${caster_radius}" h="${caster_height}" />
       </inertial>
     </link>

Commit message: Corrected wheels inertial

File: rb_theron_description/urdf/wheels/castor.urdf.xacro (robot description, xacro)
@@ -15,6 +15,6 @@
   <xacro:macro name="cylinder_inertia" params="m r h">
     <inertia  ixx="${m*(3*r*r+h*h)/12}" ixy = "0" ixz = "0"
-              iyy="${m*(3*r*r+h*h)/12}" iyz = "0"
-              izz="${m*r*r/2}" />
+              izz="${m*(3*r*r+h*h)/12}" iyz = "0"
+              iyy="${m*r*r/2}" />
   </xacro:macro>
   <xacro:macro name="caster" params="prefix parent *origin hq">

File: rb_theron_description/urdf/wheels/rubber_wheel_125.urdf.xacro (robot description, xacro)
@@ -11,5 +11,12 @@
 	<!-- in kg-->
 	<xacro:macro name="cylinder_inertia" params="m r h">
-		<inertia ixx="${m*(3*r*r+h*h)/12}" ixy = "0" ixz = "0" iyy="${m*(3*r*r+h*h)/12}" iyz = "0" izz="${m*r*r/2}" />
+		<inertia
+			iyy="${m*r*r/2}"
+			ixx="${m*(3*r*r+h*h)/12}"
+			izz="${m*(3*r*r+h*h)/12}"
+			ixy="0"
+			ixz="0"
+			iyz="0"
+		/>
 	</xacro:macro>
 	<xacro:macro name="rubber_wheel" params="prefix parent *origin reflect hq">

File: rb_theron_description/urdf/wheels/rubber_wheel_150.urdf.xacro (robot description, xacro)
@@ -11,5 +11,12 @@
 	<!-- in kg-->
 	<xacro:macro name="cylinder_inertia" params="m r h">
-		<inertia ixx="${m*(3*r*r+h*h)/12}" ixy = "0" ixz = "0" iyy="${m*(3*r*r+h*h)/12}" iyz = "0" izz="${m*r*r/2}" />
+		<inertia
+			iyy="${m*r*r/2}"
+			ixx="${m*(3*r*r+h*h)/12}"
+			izz="${m*(3*r*r+h*h)/12}"
+			ixy="0"
+			ixz="0"
+			iyz="0"
+		/>
 	</xacro:macro>
 	<xacro:macro name="rubber_wheel" params="prefix parent *origin hq">

Commit message: rb_theron_description: Set caster wheel as fixed joint

File: rb_theron_description/urdf/wheels/castor.urdf.xacro (robot description, xacro)
@@ -20,10 +20,10 @@
   <xacro:macro name="caster" params="prefix parent *origin hq">
   <!--CASTER SUPPORT -->
-  <joint name="${prefix}joint_support" type="continuous">
+  <joint name="${prefix}joint_support" type="fixed">
       <parent link="${parent}"/>
       <child link="${prefix}_support"/>
       <xacro:insert_block name="origin" />
       <axis xyz="0 0 1" rpy="0 ${M_PI} 0" />
-      <limit effort="100" velocity="100"/>
+      <!-- <limit effort="100" velocity="100"/> -->
       <!-- joint_properties damping="1.5" friction="1.5"/ -->
       <dynamics damping="0" friction="0.01"/>
@@ -55,10 +55,10 @@
  </xacro:macro>
  <xacro:macro name="caster_wheel" params="prefix parent *origin hq">
-     <joint name="${prefix}joint_wheel" type="continuous">
+     <joint name="${prefix}joint_wheel" type="fixed">
        <parent link="${parent}"/>
        <child link="${prefix}_wheel"/>
        <insert_block name="origin" />
        <axis xyz="0 1 0" rpy="0 0 0" />
-       <limit effort="100" velocity="100"/>
+       <!-- <limit effort="100" velocity="100"/> -->
        <joint_properties damping="0.1" friction="0.1"/>
     </joint>
@@ -99,5 +99,5 @@
       </inertial>
     </link>
-  <!-- Transmission is important to link the joints and the controller -->
+  <!-- Transmission is important to link the joints and the controller
     <transmission name="${prefix}_support_joint_trans">
       <type>transmission_interface/SimpleTransmission</type>
@@ -120,4 +120,5 @@
       </actuator>
     </transmission>
+  -->
     <gazebo reference="${prefix}_support">
 			<mu1 value="5.0"/>

Commit message: reverted commit caster wheels

File: rb_theron_description/urdf/wheels/castor.urdf.xacro (robot description, xacro)
@@ -18,11 +18,10 @@
               izz="${m*r*r/2}" />
   </xacro:macro>
-  <xacro:macro name="caster" params="prefix parent *origin hq use_sim">
+  <xacro:macro name="caster" params="prefix parent *origin hq">
   <!--CASTER SUPPORT -->
-  <xacro:if value="${use_sim}">
-    <joint name="${prefix}joint_support" type="continuous">
+  <joint name="${prefix}joint_support" type="continuous">
       <parent link="${parent}"/>
-      <child link="${prefix}_support"/>
-      <xacro:insert_block name="origin" />
+      <child link="${prefix}support"/>
+      <insert_block name="origin" />
       <axis xyz="0 0 1" rpy="0 ${M_PI} 0" />
       <limit effort="100" velocity="100"/>
@@ -30,17 +29,5 @@
       <dynamics damping="0" friction="0.01"/>
     </joint>
-  </xacro:if>
-  <xacro:unless value="${use_sim}">
-    <joint name="${prefix}joint_support" type="fixed">
-        <parent link="${parent}"/>
-        <child link="${prefix}_support"/>
-        <xacro:insert_block name="origin" />
-        <axis xyz="0 0 1" rpy="0 ${M_PI} 0" />
-        <!-- <limit effort="100" velocity="100"/> -->
-        <!-- joint_properties damping="1.5" friction="1.5"/ -->
-        <dynamics damping="0" friction="0.01"/>
-      </joint>
-  </xacro:unless>
-    <link name="${prefix}_support">
+    <link name="${prefix}support">
       <visual>
         <origin xyz="0 0 0" rpy="0 0 0" />
@@ -49,10 +36,10 @@
           </geometry>
       </visual>
-      <collision>
+      <!--collision>
         <origin xyz="0 0 0" rpy="0 0 0" />
           <geometry>
 	       <mesh filename="package://rb_theron_description/meshes/wheels/castor_wheel.dae" />
           </geometry>
-      </collision>
+      </collision-->
       <inertial>
         <mass value="${caster_support_mass}" />
@@ -62,31 +49,19 @@
     </link>
   <!--CASTER WHEEL -->
-  <!-- xacro:caster_wheel prefix="${prefix}" parent="${prefix}_support" hq="${hq}" -->
-  <xacro:caster_wheel prefix="${prefix}" parent="${prefix}_support" hq="${hq}" use_sim="$(arg use_sim)">
+  <!-- xacro:caster_wheel prefix="${prefix}" parent="${prefix}support" hq="${hq}" -->
+  <xacro:caster_wheel prefix="${prefix}" parent="${prefix}support" hq="${hq}">
 		<origin xyz="${caster_wheel_offset_x} ${caster_wheel_offset_y} ${caster_wheel_offset_z}" rpy="0 0 0"/>
    </xacro:caster_wheel>
  </xacro:macro>
- <xacro:macro name="caster_wheel" params="prefix parent *origin hq use_sim">
-  <xacro:if value="${use_sim}">
-    <joint name="${prefix}joint_wheel" type="continuous">
-      <parent link="${parent}"/>
-      <child link="${prefix}_wheel"/>
-      <insert_block name="origin" />
-      <axis xyz="0 1 0" rpy="0 0 0" />
-      <limit effort="100" velocity="100"/>
-      <joint_properties damping="0.1" friction="0.1"/>
-   </joint>
-  </xacro:if>
-  <xacro:unless value="${use_sim}">
-     <joint name="${prefix}joint_wheel" type="fixed">
+ <xacro:macro name="caster_wheel" params="prefix parent *origin hq">
+     <joint name="${prefix}joint_wheel" type="continuous">
        <parent link="${parent}"/>
-       <child link="${prefix}_wheel"/>
+       <child link="${prefix}wheel"/>
        <insert_block name="origin" />
        <axis xyz="0 1 0" rpy="0 0 0" />
-       <!-- <limit effort="100" velocity="100"/> -->
+       <limit effort="100" velocity="100"/>
        <joint_properties damping="0.1" friction="0.1"/>
     </joint>
-  </xacro:unless>
-    <link name="${prefix}_wheel">
+    <link name="${prefix}wheel">
       <visual>
         <!-- HIGH RESOLUTION WHEELS -->
@@ -99,5 +74,5 @@
        <!-- LOW RESOLUTION WHEELS -->
        <!-- xacro:unless value="${hq}" -->
-          <origin xyz="0 0 0" rpy="0 0 0" />
+          <origin xyz="0 0 0" rpy="${M_PI/2} 0 0" />
           <geometry>
             <cylinder length="${caster_height}" radius="${caster_radius}" />
@@ -124,28 +99,26 @@
       </inertial>
     </link>
-  <!-- Transmission is important to link the joints and the controller-->
-  <xacro:if value="${use_sim}">
-    <transmission name="${prefix}_support_joint_trans">
+  <!-- Transmission is important to link the joints and the controller -->
+    <transmission name="${prefix}support_joint_trans">
       <type>transmission_interface/SimpleTransmission</type>
       <joint name="${prefix}joint_support">
           <hardwareInterface>hardware_interface/EffortJointInterface</hardwareInterface>
       </joint>
-      <actuator name="${prefix}_support_joint_motor">
+      <actuator name="${prefix}support_joint_motor">
         <mechanicalReduction>1</mechanicalReduction>
       	<motorTorqueConstant>1</motorTorqueConstant>
       </actuator>
     </transmission>
-    <transmission name="${prefix}_wheel_joint_trans">
+    <transmission name="${prefix}wheel_joint_trans">
       <type>transmission_interface/SimpleTransmission</type>
       <joint name="${prefix}joint_wheel">
           <hardwareInterface>hardware_interface/EffortJointInterface</hardwareInterface>
       </joint>
-      <actuator name="${prefix}_wheel_joint_motor">
+      <actuator name="${prefix}wheel_joint_motor">
         <mechanicalReduction>1</mechanicalReduction>
 		<motorTorqueConstant>1</motorTorqueConstant>
       </actuator>
     </transmission>
-  </xacro:if>
-    <gazebo reference="${prefix}_support">
+    <!-- gazebo reference="${prefix}support">
 			<mu1 value="5.0"/>
 			<mu2 value="0.5"/>
@@ -154,5 +127,5 @@
 			<fdir1 value="1 0 0"/>
       <turnGravityOff>false</turnGravityOff>
-    </gazebo>
+    </gazebo -->
      <gazebo reference="${prefix}_wheel">
 			<mu1 value="100.0"/>

Commit message: Fixed problem with wheel movement. Added params for left and right wheels with the proper value in close_loop and the proper values for the PID of the joints.

File: rb_theron_description/urdf/wheels/castor.urdf.xacro (robot description, xacro)
@@ -18,16 +18,27 @@
               izz="${m*r*r/2}" />
   </xacro:macro>
-  <xacro:macro name="caster" params="prefix parent *origin hq">
+  <xacro:macro name="caster" params="prefix parent *origin hq use_sim">
   <!--CASTER SUPPORT -->
-  <joint name="${prefix}joint_support" type="continuous">
+  <xacro:if value="${use_sim}">
+    <joint name="${prefix}joint_support" type="continuous">
       <parent link="${parent}"/>
-      <child link="${prefix}support"/>
-      <insert_block name="origin" />
-      <axis xyz="0 0 1" rpy="0 ${M_PI} 0" />
-      <limit effort="100" velocity="100"/>
-      <!-- joint_properties damping="1.5" friction="1.5"/ -->
-      <dynamics damping="0" friction="0.01"/>
+      <child link="${prefix}_support"/>
+      <xacro:insert_block name="origin" />
+      <axis xyz="0 0 1" />
+      <dynamics damping="0.01" friction="0.1"/>
     </joint>
-    <link name="${prefix}support">
+  </xacro:if>
+  <xacro:unless value="${use_sim}">
+    <joint name="${prefix}joint_support" type="fixed">
+        <parent link="${parent}"/>
+        <child link="${prefix}_support"/>
+        <xacro:insert_block name="origin" />
+        <axis xyz="0 0 1" rpy="0 ${M_PI} 0" />
+        <!-- <limit effort="100" velocity="100"/> -->
+        <!-- joint_properties damping="1.5" friction="1.5"/ -->
+        <dynamics damping="0" friction="0.01"/>
+      </joint>
+  </xacro:unless>
+    <link name="${prefix}_support">
       <visual>
         <origin xyz="0 0 0" rpy="0 0 0" />
@@ -36,10 +47,4 @@
           </geometry>
       </visual>
-      <!--collision>
-        <origin xyz="0 0 0" rpy="0 0 0" />
-          <geometry>
-	       <mesh filename="package://rb_theron_description/meshes/wheels/castor_wheel.dae" />
-          </geometry>
-      </collision-->
       <inertial>
         <mass value="${caster_support_mass}" />
@@ -48,48 +53,36 @@
       </inertial>
     </link>
-  <!--CASTER WHEEL -->
-  <!-- xacro:caster_wheel prefix="${prefix}" parent="${prefix}support" hq="${hq}" -->
-  <xacro:caster_wheel prefix="${prefix}" parent="${prefix}support" hq="${hq}">
-		<origin xyz="${caster_wheel_offset_x} ${caster_wheel_offset_y} ${caster_wheel_offset_z}" rpy="0 0 0"/>
-   </xacro:caster_wheel>
- </xacro:macro>
- <xacro:macro name="caster_wheel" params="prefix parent *origin hq">
-     <joint name="${prefix}joint_wheel" type="continuous">
+    <!--CASTER WHEEL -->
+    <!-- xacro:caster_wheel prefix="${prefix}" parent="${prefix}_support" hq="${hq}" -->
+    <xacro:caster_wheel prefix="${prefix}" parent="${prefix}_support" hq="${hq}" use_sim="$(arg use_sim)">
+      <origin xyz="-0.023 ${caster_wheel_offset_y} -0.071" rpy="0 0 0" />
+    </xacro:caster_wheel>
+  </xacro:macro>
+ <xacro:macro name="caster_wheel" params="prefix parent *origin hq use_sim">
+  <xacro:if value="${use_sim}">
+    <joint name="${prefix}joint_wheel" type="continuous">
+      <parent link="${parent}"/>
+      <child link="${prefix}_wheel"/>
+      <origin xyz="-0.033 ${caster_wheel_offset_y} -0.071" rpy="0 0 0" />
+      <axis xyz="0 1 0"/>
+      <joint_properties damping="0.01" friction="0.1"/>
+   </joint>
+  </xacro:if>
+  <xacro:unless value="${use_sim}">
+     <joint name="${prefix}joint_wheel" type="fixed">
        <parent link="${parent}"/>
-       <child link="${prefix}wheel"/>
+       <child link="${prefix}_wheel"/>
        <insert_block name="origin" />
-       <axis xyz="0 1 0" rpy="0 0 0" />
-       <limit effort="100" velocity="100"/>
+       <axis xyz="0 0 1" rpy="0 0 0" />
+       <!-- <limit effort="100" velocity="100"/> -->
        <joint_properties damping="0.1" friction="0.1"/>
     </joint>
-    <link name="${prefix}wheel">
-      <visual>
-        <!-- HIGH RESOLUTION WHEELS -->
-     <!-- xacro:if value="${hq}">
-          <origin xyz="0 0 0" rpy="0 0 0" />
-          <geometry>
-		<mesh filename="package://rb_theron_description/meshes/wheels/mcq_prototype_castor_wheel.dae" />
-          </geometry>
-        </xacro:if -->
-       <!-- LOW RESOLUTION WHEELS -->
-       <!-- xacro:unless value="${hq}" -->
-          <origin xyz="0 0 0" rpy="${M_PI/2} 0 0" />
-          <geometry>
-            <cylinder length="${caster_height}" radius="${caster_radius}" />
-            <!-- sphere radius="${caster_radius}"/ -->
-          </geometry>
-        <!-- /xacro:unless -->
-      </visual>
-     <collision>
-	  <origin xyz="0 0 0" rpy="${M_PI/2} 0 0" />
-	  <!-- origin xyz="0 0 0" rpy="0 0 0" / -->
+  </xacro:unless>
+    <link name="${prefix}_wheel">
+      <collision>
+        <origin xyz="0 0 0" rpy="${M_PI/2} 0 0" />
         <geometry>
-		  <!-- mesh filename="package://rb_theron_description/meshes/wheels/mcq_prototype_castor_wheel.dae" / -->
-          <cylinder length="${caster_height}" radius="${caster_radius}" />
-          <!-- sphere radius="${caster_radius}"/ -->
+          <cylinder radius="${caster_radius}" length="${caster_height}"/>
         </geometry>
-		<surface>
-          <bounce restitution_coefficient = "1"/>
-		</surface>
       </collision>
       <inertial>
@@ -99,26 +92,28 @@
       </inertial>
     </link>
-  <!-- Transmission is important to link the joints and the controller -->
-    <transmission name="${prefix}support_joint_trans">
+  <!-- Transmission is important to link the joints and the controller-->
+  <xacro:if value="${use_sim}">
+    <transmission name="${prefix}_support_joint_trans">
       <type>transmission_interface/SimpleTransmission</type>
       <joint name="${prefix}joint_support">
           <hardwareInterface>hardware_interface/EffortJointInterface</hardwareInterface>
       </joint>
-      <actuator name="${prefix}support_joint_motor">
+      <actuator name="${prefix}_support_joint_motor">
         <mechanicalReduction>1</mechanicalReduction>
       	<motorTorqueConstant>1</motorTorqueConstant>
       </actuator>
     </transmission>
-    <transmission name="${prefix}wheel_joint_trans">
+    <transmission name="${prefix}_wheel_joint_trans">
       <type>transmission_interface/SimpleTransmission</type>
       <joint name="${prefix}joint_wheel">
           <hardwareInterface>hardware_interface/EffortJointInterface</hardwareInterface>
       </joint>
-      <actuator name="${prefix}wheel_joint_motor">
+      <actuator name="${prefix}_wheel_joint_motor">
         <mechanicalReduction>1</mechanicalReduction>
 		<motorTorqueConstant>1</motorTorqueConstant>
       </actuator>
     </transmission>
-    <!-- gazebo reference="${prefix}support">
+  </xacro:if>
+    <gazebo reference="${prefix}_support">
 			<mu1 value="5.0"/>
 			<mu2 value="0.5"/>
@@ -127,5 +122,5 @@
 			<fdir1 value="1 0 0"/>
       <turnGravityOff>false</turnGravityOff>
-    </gazebo -->
+    </gazebo>
      <gazebo reference="${prefix}_wheel">
 			<mu1 value="100.0"/>
